File: LTC3042v2.kicad_sch (KiCad schematic)
At the start: 8 parts, among them U8 LT3042EDD-PBF

Commit message: main
Connections:
- net V_12V renamed V_OUT_12V
Other:
- removed sheet LTC6655LN-5
Changed lines of the file:
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@@
-	(wire
-		(pts
-			(xy 60.96 71.12) (xy 74.93 71.12)
-		)
-		(stroke
-			(width 0)
-			(type default)
-		)
-	)
 	(wire
 		(pts
@@
 	(wire
 		(pts
-			(xy 212.09 73.66) (xy 224.79 73.66)
+			(xy 212.09 73.66) (xy 240.03 73.66)
 		)
 		(stroke
@@
 	(wire
 		(pts
+			(xy 48.26 71.12) (xy 74.93 71.12)
+		)
+		(stroke
+			(width 0)
+			(type default)
+		)
+	)
+	(wire
+		(pts
 			(xy 177.8 71.12) (xy 177.8 78.74)
 		)
@@
 		)
 	)
-	(label "V_OUT_+16.5"
-		(at 60.96 71.12 0)
+	(hierarchical_label "V_OUT_12V"
+		(shape input)
+		(at 240.03 73.66 0)
 		(effects
 			(font
 				(size 1.27 1.27)
 			)
-			(justify left bottom)
-		)
-	)
-	(label "V_12V"
-		(at 224.79 73.66 0)
+			(justify left)
+		)
+	)
+	(hierarchical_label "V_OUT_+16.5"
+		(shape input)
+		(at 48.26 71.12 180)
 		(effects
 			(font
 				(size 1.27 1.27)
 			)
-			(justify left bottom)
+			(justify right)
 		)
 	)
@@
 		(instances
 			(project "DAC11001"
-				(path "/d47dddaa-1169-4924-a666-b75ea4bc2aeb/90c28152-19e4-47c0-b14f-3d9754ce4227/da7d2b28-7b50-4d5e-9a23-a4ffde2de206"
+				(path "/d47dddaa-1169-4924-a666-b75ea4bc2aeb/c4417f33-95a3-491f-8769-9984a1736115"
 					(reference "C18")
 					(unit 1)
@@
 		(instances
 			(project "DAC11001"
-				(path "/d47dddaa-1169-4924-a666-b75ea4bc2aeb/90c28152-19e4-47c0-b14f-3d9754ce4227/da7d2b28-7b50-4d5e-9a23-a4ffde2de206"
+				(path "/d47dddaa-1169-4924-a666-b75ea4bc2aeb/c4417f33-95a3-491f-8769-9984a1736115"
 					(reference "U8")
 					(unit 1)
@@
 		(instances
 			(project "DAC11001"
-				(path "/d47dddaa-1169-4924-a666-b75ea4bc2aeb/90c28152-19e4-47c0-b14f-3d9754ce4227/da7d2b28-7b50-4d5e-9a23-a4ffde2de206"
+				(path "/d47dddaa-1169-4924-a666-b75ea4bc2aeb/c4417f33-95a3-491f-8769-9984a1736115"
 					(reference "R32")
 					(unit 1)
@@
 		(instances
 			(project "DAC11001"
-				(path "/d47dddaa-1169-4924-a666-b75ea4bc2aeb/90c28152-19e4-47c0-b14f-3d9754ce4227/da7d2b28-7b50-4d5e-9a23-a4ffde2de206"
+				(path "/d47dddaa-1169-4924-a666-b75ea4bc2aeb/c4417f33-95a3-491f-8769-9984a1736115"
 					(reference "R23")
 					(unit 1)
@@
 		(instances
 			(project "DAC11001"
-				(path "/d47dddaa-1169-4924-a666-b75ea4bc2aeb/90c28152-19e4-47c0-b14f-3d9754ce4227/da7d2b28-7b50-4d5e-9a23-a4ffde2de206"
+				(path "/d47dddaa-1169-4924-a666-b75ea4bc2aeb/c4417f33-95a3-491f-8769-9984a1736115"
 					(reference "#PWR037")
 					(unit 1)
@@
 		(instances
 			(project "DAC11001"
-				(path "/d47dddaa-1169-4924-a666-b75ea4bc2aeb/90c28152-19e4-47c0-b14f-3d9754ce4227/da7d2b28-7b50-4d5e-9a23-a4ffde2de206"
+				(path "/d47dddaa-1169-4924-a666-b75ea4bc2aeb/c4417f33-95a3-491f-8769-9984a1736115"
 					(reference "R33")
 					(unit 1)
@@
 		(instances
 			(project "DAC11001"
-				(path "/d47dddaa-1169-4924-a666-b75ea4bc2aeb/90c28152-19e4-47c0-b14f-3d9754ce4227/da7d2b28-7b50-4d5e-9a23-a4ffde2de206"
+				(path "/d47dddaa-1169-4924-a666-b75ea4bc2aeb/c4417f33-95a3-491f-8769-9984a1736115"
 					(reference "R34")
 					(unit 1)
@@
 		(instances
 			(project "DAC11001"
-				(path "/d47dddaa-1169-4924-a666-b75ea4bc2aeb/90c28152-19e4-47c0-b14f-3d9754ce4227/da7d2b28-7b50-4d5e-9a23-a4ffde2de206"
+				(path "/d47dddaa-1169-4924-a666-b75ea4bc2aeb/c4417f33-95a3-491f-8769-9984a1736115"
 					(reference "C17")
 					(unit 1)
@@
 		(instances
 			(project "DAC11001"
-				(path "/d47dddaa-1169-4924-a666-b75ea4bc2aeb/90c28152-19e4-47c0-b14f-3d9754ce4227/da7d2b28-7b50-4d5e-9a23-a4ffde2de206"
+				(path "/d47dddaa-1169-4924-a666-b75ea4bc2aeb/c4417f33-95a3-491f-8769-9984a1736115"
 					(reference "C38")
 					(unit 1)
 				)
 			)
-		)
-	)
-	(sheet
-		(at 19.05 21.59)
-		(size 27.94 8.89)
-		(exclude_from_sim no)
-		(in_bom yes)
-		(on_board yes)
-		(dnp no)
-		(fields_autoplaced yes)
-		(stroke
-			(width 0.1524)
-			(type solid)
-		)
-		(fill
-			(color 0 0 0 0)
-		)
-		(property "Sheetname" "LTC6655LN-5"
-			(at 19.05 20.8784 0)
-			(show_name no)
-			(do_not_autoplace no)
-			(effects
-				(font
-					(size 1.27 1.27)
-				)
-				(justify left bottom)
-			)
-		)
-		(property "Sheetfile" "ltc6655ln-5.kicad_sch"
-			(at 19.05 31.0646 0)
-			(show_name no)
-			(do_not_autoplace no)
-			(effects
-				(font
-					(size 1.27 1.27)
-				)
-				(justify left top)
-			)
-		)
-		(instances
-			(project "DAC11001"
-				(path "/d47dddaa-1169-4924-a666-b75ea4bc2aeb/90c28152-19e4-47c0-b14f-3d9754ce4227/da7d2b28-7b50-4d5e-9a23-a4ffde2de206"
-					(page "3")
-				)
-			)
