File: ltc6655ln-5_1.kicad_sch (KiCad schematic)
At the start: 2 parts, among them U5 LTC6655LNCHMS8-5-PBF

Commit message: main
Connections:
- net V_12V renamed V_OUT_12V
Other:
- removed sheet OPA828_4X
