File: iso7761.kicad_sch (KiCad schematic)
At the start: 1 part, among them U6 ISO7761DW

Commit message: modular
Changed lines of the file:
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@@
 	(wire
 		(pts
-			(xy 124.46 59.69) (xy 151.13 59.69)
-		)
-		(stroke
-			(width 0)
-			(type default)
-		)
-	)
-	(wire
-		(pts
-			(xy 124.46 80.01) (xy 151.13 80.01)
-		)
-		(stroke
-			(width 0)
-			(type default)
-		)
-	)
-	(wire
-		(pts
-			(xy 124.46 85.09) (xy 151.13 85.09)
-		)
-		(stroke
-			(width 0)
-			(type default)
-		)
-	)
-	(wire
-		(pts
-			(xy 124.46 64.77) (xy 151.13 64.77)
-		)
-		(stroke
-			(width 0)
-			(type default)
-		)
-	)
-	(wire
-		(pts
-			(xy 124.46 74.93) (xy 151.13 74.93)
-		)
-		(stroke
-			(width 0)
-			(type default)
-		)
-	)
-	(wire
-		(pts
-			(xy 124.46 69.85) (xy 151.13 69.85)
-		)
-		(stroke
-			(width 0)
-			(type default)
+			(xy 109.22 92.71) (xy 115.57 92.71)
+		)
+		(stroke
+			(width 0)
+			(type default)
+		)
+	)
+	(wire
+		(pts
+			(xy 109.22 77.47) (xy 115.57 77.47)
+		)
+		(stroke
+			(width 0)
+			(type default)
+		)
+	)
+	(wire
+		(pts
+			(xy 109.22 97.79) (xy 115.57 97.79)
+		)
+		(stroke
+			(width 0)
+			(type default)
+		)
+	)
+	(wire
+		(pts
+			(xy 109.22 72.39) (xy 115.57 72.39)
+		)
+		(stroke
+			(width 0)
+			(type default)
+		)
+	)
+	(wire
+		(pts
+			(xy 109.22 87.63) (xy 115.57 87.63)
+		)
+		(stroke
+			(width 0)
+			(type default)
+		)
+	)
+	(wire
+		(pts
+			(xy 109.22 82.55) (xy 115.57 82.55)
+		)
+		(stroke
+			(width 0)
+			(type default)
+		)
+	)
+	(label "SDO"
+		(at 115.57 97.79 0)
+		(effects
+			(font
+				(size 1.27 1.27)
+			)
+			(justify left bottom)
+		)
+	)
+	(label "CLR"
+		(at 115.57 87.63 0)
+		(effects
+			(font
+				(size 1.27 1.27)
+			)
+			(justify left bottom)
 		)
 	)
 	(label "SYNC"
-		(at 151.13 59.69 0)
-		(effects
-			(font
-				(size 1.27 1.27)
-			)
-			(justify left bottom)
-		)
-	)
-	(label "SDO"
-		(at 151.13 85.09 0)
+		(at 115.57 72.39 0)
 		(effects
 			(font
@@
 	)
 	(label "SCLK"
-		(at 151.13 69.85 0)
-		(effects
-			(font
-				(size 1.27 1.27)
-			)
-			(justify left bottom)
-		)
-	)
-	(label "CLR"
-		(at 151.13 74.93 0)
+		(at 115.57 82.55 0)
 		(effects
 			(font
@@
 	)
 	(label "SDIN"
-		(at 151.13 64.77 0)
+		(at 115.57 77.47 0)
 		(effects
 			(font
@@
 	)
 	(label "LDAC"
-		(at 151.13 80.01 0)
+		(at 115.57 92.71 0)
 		(effects
 			(font
@@
 	(symbol
 		(lib_id "2026-07-13_21-09-16:ISO7761DW")
-		(at 104.14 72.39 0)
+		(at 88.9 85.09 0)
 		(unit 1)
 		(body_style 1)
@@
 		(fields_autoplaced yes)
 		(property "Reference" "U6"
-			(at 104.14 44.45 0)
+			(at 88.9 57.15 0)
 			(show_name no)
 			(do_not_autoplace no)
@@
 		)
 		(property "Value" "ISO7761DW"
-			(at 104.14 46.99 0)
+			(at 88.9 59.69 0)
 			(show_name no)
 			(do_not_autoplace no)
@@
 		)
 		(property "Footprint" "DW0016B_N"
-			(at 104.14 72.39 0)
+			(at 88.9 85.09 0)
 			(hide yes)
 			(show_name no)
@@
 		)
 		(property "Datasheet" "https://www.ti.com/lit/gpn/iso7761"
-			(at 104.14 72.39 0)
+			(at 88.9 85.09 0)
 			(hide yes)
 			(show_name no)
@@
 		)
 		(property "Description" ""
-			(at 104.14 72.39 0)
+			(at 88.9 85.09 0)
 			(hide yes)
 			(show_name no)
@@
 		(instances
 			(project "DAC11001"
-				(path "/d47dddaa-1169-4924-a666-b75ea4bc2aeb/7bb55e9d-69bb-475a-95aa-ce084c4b1842/a215338a-5bae-4d4e-9d14-5380f08ccb1a"
+				(path "/7d6a26c1-172d-4ef1-b333-30f014f26d9e"
 					(reference "U6")
 					(unit 1)
@@
 		)
 	)
+	(sheet_instances
+		(path "/"
+			(page "10")
+		)
+	)
+	(embedded_fonts no)
 )
