File: lt3042.kicad_sch (KiCad schematic)
At the start: 8 parts, among them U3 LT3042EDD-PBF

Commit message: main
Changed lines of the file:
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@@
+	)
+	(junction
+		(at 96.52 71.12)
+		(diameter 0)
+		(color 0 0 0 0)
 	)
 	(junction
@@
 	)
 	(junction
-		(at 96.52 71.12)
-		(diameter 0)
-		(color 0 0 0 0)
-	)
-	(junction
 		(at 184.15 73.66)
 		(diameter 0)
@@
 	(wire
 		(pts
-			(xy 82.55 71.12) (xy 96.52 71.12)
+			(xy 81.28 71.12) (xy 96.52 71.12)
 		)
 		(stroke
@@
 		)
 	)
-	(label "V_OUT_+16.5"
-		(at 82.55 71.12 0)
-		(effects
-			(font
-				(size 1.27 1.27)
-			)
-			(justify left bottom)
-		)
-	)
-	(label "V_C_+15V"
+	(hierarchical_label "V_C_+15V"
+		(shape input)
 		(at 246.38 73.66 0)
 		(effects
@@
 				(size 1.27 1.27)
 			)
-			(justify left bottom)
-		)
-	)
+			(justify left)
+		)
+	)
+	(hierarchical_label "V_OUT_+16.5"
+		(shape input)
+		(at 81.28 71.12 180)
+		(effects
+			(font
+				(size 1.27 1.27)
+			)
+			(justify right)
+		)
+	)

Commit message: main
Parts:
- C6: value C -> C2
Changed lines of the file:
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@@
 		(instances
 			(project "DAC11001"
-				(path "/d47dddaa-1169-4924-a666-b75ea4bc2aeb/5ad28e6f-ee73-4b65-bae6-2cd262b8ea89/674a7779-f709-41a4-ab06-7cf143a54cee/e1ae31ad-1dac-4987-a3d4-790585f171d3"
+				(path "/d47dddaa-1169-4924-a666-b75ea4bc2aeb/7e4ac72e-4486-470f-b637-0752120cc81e"
+					(reference "R21")
+					(unit 1)
+				)
+			)
+			(project "DAC11001"
+				(path "/e0aa5e38-0527-4cf2-b522-8958e99675c0/a51504ea-beb4-463b-b6c9-172c1b9f5f4b"
 					(reference "R6")
 					(unit 1)
@@
 		(instances
 			(project "DAC11001"
-				(path "/d47dddaa-1169-4924-a666-b75ea4bc2aeb/5ad28e6f-ee73-4b65-bae6-2cd262b8ea89/674a7779-f709-41a4-ab06-7cf143a54cee/e1ae31ad-1dac-4987-a3d4-790585f171d3"
+				(path "/d47dddaa-1169-4924-a666-b75ea4bc2aeb/7e4ac72e-4486-470f-b637-0752120cc81e"
+					(reference "R19")
+					(unit 1)
+				)
+			)
+			(project "DAC11001"
+				(path "/e0aa5e38-0527-4cf2-b522-8958e99675c0/a51504ea-beb4-463b-b6c9-172c1b9f5f4b"
 					(reference "R4")
 					(unit 1)
@@
 		(instances
 			(project "DAC11001"
-				(path "/d47dddaa-1169-4924-a666-b75ea4bc2aeb/5ad28e6f-ee73-4b65-bae6-2cd262b8ea89/674a7779-f709-41a4-ab06-7cf143a54cee/e1ae31ad-1dac-4987-a3d4-790585f171d3"
+				(path "/d47dddaa-1169-4924-a666-b75ea4bc2aeb/7e4ac72e-4486-470f-b637-0752120cc81e"
+					(reference "R22")
+					(unit 1)
+				)
+			)
+			(project "DAC11001"
+				(path "/e0aa5e38-0527-4cf2-b522-8958e99675c0/a51504ea-beb4-463b-b6c9-172c1b9f5f4b"
 					(reference "R7")
 					(unit 1)
@@
 		(dnp no)
 		(fields_autoplaced yes)
-		(property "Reference" "#PWR019"
+		(property "Reference" "#PWR038"
 			(at 162.56 113.03 0)
 			(hide yes)
@@
 		(instances
 			(project "DAC11001"
-				(path "/d47dddaa-1169-4924-a666-b75ea4bc2aeb/5ad28e6f-ee73-4b65-bae6-2cd262b8ea89/674a7779-f709-41a4-ab06-7cf143a54cee/e1ae31ad-1dac-4987-a3d4-790585f171d3"
+				(path "/d47dddaa-1169-4924-a666-b75ea4bc2aeb/7e4ac72e-4486-470f-b637-0752120cc81e"
 					(reference "#PWR019")
+					(unit 1)
+				)
+			)
+			(project "DAC11001"
+				(path "/e0aa5e38-0527-4cf2-b522-8958e99675c0/a51504ea-beb4-463b-b6c9-172c1b9f5f4b"
+					(reference "#PWR038")
 					(unit 1)
 				)
@@
 		(instances
 			(project "DAC11001"
-				(path "/d47dddaa-1169-4924-a666-b75ea4bc2aeb/5ad28e6f-ee73-4b65-bae6-2cd262b8ea89/674a7779-f709-41a4-ab06-7cf143a54cee/e1ae31ad-1dac-4987-a3d4-790585f171d3"
+				(path "/d47dddaa-1169-4924-a666-b75ea4bc2aeb/7e4ac72e-4486-470f-b637-0752120cc81e"
+					(reference "U9")
+					(unit 1)
+				)
+			)
+			(project "DAC11001"
+				(path "/e0aa5e38-0527-4cf2-b522-8958e99675c0/a51504ea-beb4-463b-b6c9-172c1b9f5f4b"
 					(reference "U3")
 					(unit 1)
@@
 		(instances
 			(project "DAC11001"
-				(path "/d47dddaa-1169-4924-a666-b75ea4bc2aeb/5ad28e6f-ee73-4b65-bae6-2cd262b8ea89/674a7779-f709-41a4-ab06-7cf143a54cee/e1ae31ad-1dac-4987-a3d4-790585f171d3"
+				(path "/d47dddaa-1169-4924-a666-b75ea4bc2aeb/7e4ac72e-4486-470f-b637-0752120cc81e"
+					(reference "R20")
+					(unit 1)
+				)
+			)
+			(project "DAC11001"
+				(path "/e0aa5e38-0527-4cf2-b522-8958e99675c0/a51504ea-beb4-463b-b6c9-172c1b9f5f4b"
 					(reference "R5")
 					(unit 1)
@@
 		(instances
 			(project "DAC11001"
-				(path "/d47dddaa-1169-4924-a666-b75ea4bc2aeb/5ad28e6f-ee73-4b65-bae6-2cd262b8ea89/674a7779-f709-41a4-ab06-7cf143a54cee/e1ae31ad-1dac-4987-a3d4-790585f171d3"
+				(path "/d47dddaa-1169-4924-a666-b75ea4bc2aeb/7e4ac72e-4486-470f-b637-0752120cc81e"
+					(reference "C15")
+					(unit 1)
+				)
+			)
+			(project "DAC11001"
+				(path "/e0aa5e38-0527-4cf2-b522-8958e99675c0/a51504ea-beb4-463b-b6c9-172c1b9f5f4b"
 					(reference "C5")
 					(unit 1)
@@
 			)
 		)
-		(property "Value" "C"
+		(property "Value" "C2"
 			(at 237.49 88.8999 0)
 			(show_name no)
@@
 		(instances
 			(project "DAC11001"
-				(path "/d47dddaa-1169-4924-a666-b75ea4bc2aeb/5ad28e6f-ee73-4b65-bae6-2cd262b8ea89/674a7779-f709-41a4-ab06-7cf143a54cee/e1ae31ad-1dac-4987-a3d4-790585f171d3"
+				(path "/d47dddaa-1169-4924-a666-b75ea4bc2aeb/7e4ac72e-4486-470f-b637-0752120cc81e"
+					(reference "C16")
+					(unit 1)
+				)
+			)
+			(project "DAC11001"
+				(path "/e0aa5e38-0527-4cf2-b522-8958e99675c0/a51504ea-beb4-463b-b6c9-172c1b9f5f4b"
 					(reference "C6")
 					(unit 1)
@@
 		(instances
 			(project "DAC11001"
-				(path "/d47dddaa-1169-4924-a666-b75ea4bc2aeb/5ad28e6f-ee73-4b65-bae6-2cd262b8ea89/674a7779-f709-41a4-ab06-7cf143a54cee/e1ae31ad-1dac-4987-a3d4-790585f171d3"
+				(path "/d47dddaa-1169-4924-a666-b75ea4bc2aeb/7e4ac72e-4486-470f-b637-0752120cc81e"
+					(reference "C14")
+					(unit 1)
+				)
+			)
+			(project "DAC11001"
+				(path "/e0aa5e38-0527-4cf2-b522-8958e99675c0/a51504ea-beb4-463b-b6c9-172c1b9f5f4b"
 					(reference "C4")
 					(unit 1)

Commit message: modular
Connections:
- net V_C_+15V renamed V_P_C_+15V
- net V_OUT_+16.5 renamed V_P_+16.5V
