File: lt3042.kicad_sch (KiCad schematic)
At the start: 8 parts, among them U3 LT3042EDD-PBF

Commit message: globaled
Changed lines of the file:
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@@
+	)
+	(junction
+		(at 189.23 83.82)
+		(diameter 0)
+		(color 0 0 0 0)
+	)
+	(junction
+		(at 180.34 96.52)
+		(diameter 0)
+		(color 0 0 0 0)
+	)
+	(junction
+		(at 86.36 76.2)
+		(diameter 0)
+		(color 0 0 0 0)
+	)
+	(junction
+		(at 152.4 111.76)
+		(diameter 0)
+		(color 0 0 0 0)
+	)
+	(junction
+		(at 173.99 78.74)
+		(diameter 0)
+		(color 0 0 0 0)
+	)
+	(junction
+		(at 105.41 78.74)
+		(diameter 0)
+		(color 0 0 0 0)
 	)
 	(junction
@@
 	)
 	(junction
-		(at 189.23 83.82)
-		(diameter 0)
-		(color 0 0 0 0)
-	)
-	(junction
-		(at 180.34 96.52)
-		(diameter 0)
-		(color 0 0 0 0)
-	)
-	(junction
-		(at 86.36 76.2)
-		(diameter 0)
-		(color 0 0 0 0)
-	)
-	(junction
-		(at 152.4 111.76)
-		(diameter 0)
-		(color 0 0 0 0)
-	)
-	(junction
-		(at 173.99 78.74)
-		(diameter 0)
-		(color 0 0 0 0)
-	)
-	(junction
-		(at 105.41 78.74)
-		(diameter 0)
-		(color 0 0 0 0)
-	)
-	(junction
 		(at 180.34 104.14)
 		(diameter 0)
@@
 	(wire
 		(pts
-			(xy 223.52 78.74) (xy 236.22 78.74)
+			(xy 223.52 78.74) (xy 255.27 78.74)
 		)
 		(stroke
@@
 		)
 	)
-	(label "V_P_C_+15V"
-		(at 236.22 78.74 0)
+	(global_label "V_P_C_+15V"
+		(shape input)
+		(at 255.27 78.74 0)
+		(fields_autoplaced yes)
 		(effects
 			(font
 				(size 1.27 1.27)
 			)
-			(justify left bottom)
-		)
-	)
-	(label "V_P_+16.5V"
-		(at 71.12 76.2 0)
+			(justify left)
+		)
+		(property "Intersheetrefs" "${INTERSHEET_REFS}"
+			(at 269.8666 78.74 0)
+			(hide yes)
+			(show_name no)
+			(do_not_autoplace no)
+			(effects
+				(font
+					(size 1.27 1.27)
+				)
+				(justify left)
+			)
+		)
+	)
+	(global_label "V_P_+16.5V"
+		(shape input)
+		(at 71.12 76.2 180)
+		(fields_autoplaced yes)
 		(effects
 			(font
 				(size 1.27 1.27)
 			)
-			(justify left bottom)
+			(justify right)
+		)
+		(property "Intersheetrefs" "${INTERSHEET_REFS}"
+			(at 56.9467 76.2 0)
+			(hide yes)
+			(show_name no)
+			(do_not_autoplace no)
+			(effects
+				(font
+					(size 1.27 1.27)
+				)
+				(justify right)
+			)
 		)
 	)
@@
 				)
 			)
-			(project "DAC11001"
-				(path "/d47dddaa-1169-4924-a666-b75ea4bc2aeb/36834370-2082-4f70-b859-136ec9471013"
-					(reference "U10")
-					(unit 1)
-				)
-			)
 		)
 	)
@@
 				)
 			)
-			(project "DAC11001"
-				(path "/d47dddaa-1169-4924-a666-b75ea4bc2aeb/36834370-2082-4f70-b859-136ec9471013"
-					(reference "R44")
-					(unit 1)
-				)
-			)
 		)
 	)
@@
 				)
 			)
-			(project "DAC11001"
-				(path "/d47dddaa-1169-4924-a666-b75ea4bc2aeb/36834370-2082-4f70-b859-136ec9471013"
-					(reference "C42")
-					(unit 1)
-				)
-			)
 		)
 	)
@@
 				)
 			)
-			(project "DAC11001"
-				(path "/d47dddaa-1169-4924-a666-b75ea4bc2aeb/36834370-2082-4f70-b859-136ec9471013"
-					(reference "#PWR038")
-					(unit 1)
-				)
-			)
 		)
 	)
@@
 				)
 			)
-			(project "DAC11001"
-				(path "/d47dddaa-1169-4924-a666-b75ea4bc2aeb/36834370-2082-4f70-b859-136ec9471013"
-					(reference "R45")
-					(unit 1)
-				)
-			)
 		)
 	)
@@
 				)
 			)
-			(project "DAC11001"
-				(path "/d47dddaa-1169-4924-a666-b75ea4bc2aeb/36834370-2082-4f70-b859-136ec9471013"
-					(reference "R46")
-					(unit 1)
-				)
-			)
 		)
 	)
@@
 				)
 			)
-			(project "DAC11001"
-				(path "/d47dddaa-1169-4924-a666-b75ea4bc2aeb/36834370-2082-4f70-b859-136ec9471013"
-					(reference "C40")
-					(unit 1)
-				)
-			)
 		)
 	)
@@
 				)
 			)
-			(project "DAC11001"
-				(path "/d47dddaa-1169-4924-a666-b75ea4bc2aeb/36834370-2082-4f70-b859-136ec9471013"
-					(reference "C41")
-					(unit 1)
-				)
-			)
 		)
 	)
@@
 				)
 			)
-			(project "DAC11001"
-				(path "/d47dddaa-1169-4924-a666-b75ea4bc2aeb/36834370-2082-4f70-b859-136ec9471013"
-					(reference "R43")
-					(unit 1)
-				)
-			)
-		)
-	)
-	(sheet_instances
-		(path "/"
-			(page "2")
-		)
-	)
+		)
+	)

Commit message: done
Parts:
- renumbered C4 to C45, C5 to C46, C6 to C47, R4 to R47, R5 to R48, R6 to R49, R7 to R50, U3 to U15
Changed lines of the file:
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@@
 		(dnp no)
 		(fields_autoplaced yes)
-		(property "Reference" "U3"
+		(property "Reference" "U15"
 			(at 143.51 66.04 0)
 			(show_name no)
@@
 		(instances
 			(project "DAC11001"
+				(path "/688e2b68-3871-489b-b27a-c18d3c11fcf6/1cdb1a95-8826-45a6-bddc-c4b97ae2a13e"
+					(reference "U1")
+					(unit 1)
+				)
+			)
+			(project "DAC11001"
 				(path "/924ca917-6b99-40f8-9087-94374e4e1bff"
 					(reference "U3")
+					(unit 1)
+				)
+			)
+			(project "DAC11001"
+				(path "/d47dddaa-1169-4924-a666-b75ea4bc2aeb/a8da5177-43c4-4665-b682-d49b9fc3d5b2/1cdb1a95-8826-45a6-bddc-c4b97ae2a13e"
+					(reference "U15")
 					(unit 1)
 				)
@@
 		(dnp no)
 		(fields_autoplaced yes)
-		(property "Reference" "R5"
+		(property "Reference" "R48"
 			(at 186.69 99.0599 0)
 			(show_name no)
@@
 		(instances
 			(project "DAC11001"
+				(path "/688e2b68-3871-489b-b27a-c18d3c11fcf6/1cdb1a95-8826-45a6-bddc-c4b97ae2a13e"
+					(reference "R20")
+					(unit 1)
+				)
+			)
+			(project "DAC11001"
 				(path "/924ca917-6b99-40f8-9087-94374e4e1bff"
 					(reference "R5")
+					(unit 1)
+				)
+			)
+			(project "DAC11001"
+				(path "/d47dddaa-1169-4924-a666-b75ea4bc2aeb/a8da5177-43c4-4665-b682-d49b9fc3d5b2/1cdb1a95-8826-45a6-bddc-c4b97ae2a13e"
+					(reference "R48")
 					(unit 1)
 				)
@@
 		(dnp no)
 		(fields_autoplaced yes)
-		(property "Reference" "C6"
+		(property "Reference" "C47"
 			(at 227.33 91.4399 0)
 			(show_name no)
@@
 		(instances
 			(project "DAC11001"
+				(path "/688e2b68-3871-489b-b27a-c18d3c11fcf6/1cdb1a95-8826-45a6-bddc-c4b97ae2a13e"
+					(reference "C16")
+					(unit 1)
+				)
+			)
+			(project "DAC11001"
 				(path "/924ca917-6b99-40f8-9087-94374e4e1bff"
 					(reference "C6")
+					(unit 1)
+				)
+			)
+			(project "DAC11001"
+				(path "/d47dddaa-1169-4924-a666-b75ea4bc2aeb/a8da5177-43c4-4665-b682-d49b9fc3d5b2/1cdb1a95-8826-45a6-bddc-c4b97ae2a13e"
+					(reference "C47")
 					(unit 1)
 				)
@@
 		(instances
 			(project "DAC11001"
+				(path "/688e2b68-3871-489b-b27a-c18d3c11fcf6/1cdb1a95-8826-45a6-bddc-c4b97ae2a13e"
+					(reference "#PWR038")
+					(unit 1)
+				)
+			)
+			(project "DAC11001"
 				(path "/924ca917-6b99-40f8-9087-94374e4e1bff"
+					(reference "#PWR038")
+					(unit 1)
+				)
+			)
+			(project "DAC11001"
+				(path "/d47dddaa-1169-4924-a666-b75ea4bc2aeb/a8da5177-43c4-4665-b682-d49b9fc3d5b2/1cdb1a95-8826-45a6-bddc-c4b97ae2a13e"
 					(reference "#PWR038")
 					(unit 1)
@@
 		(dnp no)
 		(fields_autoplaced yes)
-		(property "Reference" "R6"
+		(property "Reference" "R49"
 			(at 210.82 83.8199 0)
 			(show_name no)
@@
 		(instances
 			(project "DAC11001"
+				(path "/688e2b68-3871-489b-b27a-c18d3c11fcf6/1cdb1a95-8826-45a6-bddc-c4b97ae2a13e"
+					(reference "R21")
+					(unit 1)
+				)
+			)
+			(project "DAC11001"
 				(path "/924ca917-6b99-40f8-9087-94374e4e1bff"
 					(reference "R6")
+					(unit 1)
+				)
+			)
+			(project "DAC11001"
+				(path "/d47dddaa-1169-4924-a666-b75ea4bc2aeb/a8da5177-43c4-4665-b682-d49b9fc3d5b2/1cdb1a95-8826-45a6-bddc-c4b97ae2a13e"
+					(reference "R49")
 					(unit 1)
 				)
@@
 		(dnp no)
 		(fields_autoplaced yes)
-		(property "Reference" "R7"
+		(property "Reference" "R50"
 			(at 210.82 93.9799 0)
 			(show_name no)
@@
 		(instances
 			(project "DAC11001"
+				(path "/688e2b68-3871-489b-b27a-c18d3c11fcf6/1cdb1a95-8826-45a6-bddc-c4b97ae2a13e"
+					(reference "R22")
+					(unit 1)
+				)
+			)
+			(project "DAC11001"
 				(path "/924ca917-6b99-40f8-9087-94374e4e1bff"
 					(reference "R7")
+					(unit 1)
+				)
+			)
+			(project "DAC11001"
+				(path "/d47dddaa-1169-4924-a666-b75ea4bc2aeb/a8da5177-43c4-4665-b682-d49b9fc3d5b2/1cdb1a95-8826-45a6-bddc-c4b97ae2a13e"
+					(reference "R50")
 					(unit 1)
 				)
@@
 		(dnp no)
 		(fields_autoplaced yes)
-		(property "Reference" "C4"
+		(property "Reference" "C45"
 			(at 90.17 78.7399 0)
 			(show_name no)
@@
 		(instances
 			(project "DAC11001"
+				(path "/688e2b68-3871-489b-b27a-c18d3c11fcf6/1cdb1a95-8826-45a6-bddc-c4b97ae2a13e"
+					(reference "C14")
+					(unit 1)
+				)
+			)
+			(project "DAC11001"
 				(path "/924ca917-6b99-40f8-9087-94374e4e1bff"
 					(reference "C4")
+					(unit 1)
+				)
+			)
+			(project "DAC11001"
+				(path "/d47dddaa-1169-4924-a666-b75ea4bc2aeb/a8da5177-43c4-4665-b682-d49b9fc3d5b2/1cdb1a95-8826-45a6-bddc-c4b97ae2a13e"
+					(reference "C45")
 					(unit 1)
 				)
@@
 		(dnp no)
 		(fields_autoplaced yes)
-		(property "Reference" "C5"
+		(property "Reference" "C46"
 			(at 179.07 99.0599 0)
 			(show_name no)
@@
 		(instances
 			(project "DAC11001"
+				(path "/688e2b68-3871-489b-b27a-c18d3c11fcf6/1cdb1a95-8826-45a6-bddc-c4b97ae2a13e"
+					(reference "C15")
+					(unit 1)
+				)
+			)
+			(project "DAC11001"
 				(path "/924ca917-6b99-40f8-9087-94374e4e1bff"
 					(reference "C5")
+					(unit 1)
+				)
+			)
+			(project "DAC11001"
+				(path "/d47dddaa-1169-4924-a666-b75ea4bc2aeb/a8da5177-43c4-4665-b682-d49b9fc3d5b2/1cdb1a95-8826-45a6-bddc-c4b97ae2a13e"
+					(reference "C46")
 					(unit 1)
 				)
@@
 		(dnp no)
 		(fields_autoplaced yes)
-		(property "Reference" "R4"
+		(property "Reference" "R47"
 			(at 115.57 100.3299 0)
 			(show_name no)
@@
 		(instances
 			(project "DAC11001"
+				(path "/688e2b68-3871-489b-b27a-c18d3c11fcf6/1cdb1a95-8826-45a6-bddc-c4b97ae2a13e"
+					(reference "R19")
+					(unit 1)
+				)
+			)
+			(project "DAC11001"
 				(path "/924ca917-6b99-40f8-9087-94374e4e1bff"
 					(reference "R4")
 					(unit 1)
 				)
+			)
+			(project "DAC11001"
+				(path "/d47dddaa-1169-4924-a666-b75ea4bc2aeb/a8da5177-43c4-4665-b682-d49b9fc3d5b2/1cdb1a95-8826-45a6-bddc-c4b97ae2a13e"
+					(reference "R47")
+					(unit 1)
+				)
