File: lt3042v2.kicad_sch (KiCad schematic)
At the start: 8 parts, among them U8 LT3042EDD-PBF

Commit message: modular
Connections:
- net V_OUT_+16.5 renamed V_P_+16.5V
- net V_OUT_12V renamed V_P_+12V
