File: lt3042v2.kicad_sch (KiCad schematic)
At the start: 8 parts, among them U8 LT3042EDD-PBF

Commit message: globaled
Changed lines of the file:
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@@
 		)
 	)
-	(label "V_P_+12V"
+	(global_label "V_P_+12V"
+		(shape input)
 		(at 236.22 80.01 0)
+		(fields_autoplaced yes)
 		(effects
 			(font
 				(size 1.27 1.27)
 			)
-			(justify left bottom)
-		)
-	)
-	(label "V_P_+16.5V"
-		(at 44.45 77.47 0)
+			(justify left)
+		)
+		(property "Intersheetrefs" "${INTERSHEET_REFS}"
+			(at 248.579 80.01 0)
+			(hide yes)
+			(show_name no)
+			(do_not_autoplace no)
+			(effects
+				(font
+					(size 1.27 1.27)
+				)
+				(justify left)
+			)
+		)
+	)
+	(global_label "V_P_+16.5V"
+		(shape input)
+		(at 44.45 77.47 180)
+		(fields_autoplaced yes)
 		(effects
 			(font
 				(size 1.27 1.27)
 			)
-			(justify left bottom)
+			(justify right)
+		)
+		(property "Intersheetrefs" "${INTERSHEET_REFS}"
+			(at 30.2767 77.47 0)
+			(hide yes)
+			(show_name no)
+			(do_not_autoplace no)
+			(effects
+				(font
+					(size 1.27 1.27)
+				)
+				(justify right)
+			)
 		)
 	)
@@
 				)
 			)
-			(project "DAC11001"
-				(path "/d47dddaa-1169-4924-a666-b75ea4bc2aeb/b0c6e875-56fd-4a79-9737-deb22c9bb7f9"
-					(reference "R52")
-					(unit 1)
-				)
-			)
 		)
 	)
@@
 				)
 			)
-			(project "DAC11001"
-				(path "/d47dddaa-1169-4924-a666-b75ea4bc2aeb/b0c6e875-56fd-4a79-9737-deb22c9bb7f9"
-					(reference "C46")
-					(unit 1)
-				)
-			)
 		)
 	)
@@
 				)
 			)
-			(project "DAC11001"
-				(path "/d47dddaa-1169-4924-a666-b75ea4bc2aeb/b0c6e875-56fd-4a79-9737-deb22c9bb7f9"
-					(reference "R51")
-					(unit 1)
-				)
-			)
 		)
 	)
@@
 				)
 			)
-			(project "DAC11001"
-				(path "/d47dddaa-1169-4924-a666-b75ea4bc2aeb/b0c6e875-56fd-4a79-9737-deb22c9bb7f9"
-					(reference "U16")
-					(unit 1)
-				)
-			)
 		)
 	)
@@
 				)
 			)
-			(project "DAC11001"
-				(path "/d47dddaa-1169-4924-a666-b75ea4bc2aeb/b0c6e875-56fd-4a79-9737-deb22c9bb7f9"
-					(reference "R54")
-					(unit 1)
-				)
-			)
 		)
 	)
@@
 				)
 			)
-			(project "DAC11001"
-				(path "/d47dddaa-1169-4924-a666-b75ea4bc2aeb/b0c6e875-56fd-4a79-9737-deb22c9bb7f9"
-					(reference "C48")
-					(unit 1)
-				)
-			)
 		)
 	)
@@
 				)
 			)
-			(project "DAC11001"
-				(path "/d47dddaa-1169-4924-a666-b75ea4bc2aeb/b0c6e875-56fd-4a79-9737-deb22c9bb7f9"
-					(reference "C47")
-					(unit 1)
-				)
-			)
 		)
 	)
@@
 				)
 			)
-			(project "DAC11001"
-				(path "/d47dddaa-1169-4924-a666-b75ea4bc2aeb/b0c6e875-56fd-4a79-9737-deb22c9bb7f9"
-					(reference "R53")
-					(unit 1)
-				)
-			)
 		)
 	)
@@
 					(reference "#PWR037")
 					(unit 1)
-				)
-			)
-			(project "DAC11001"
-				(path "/d47dddaa-1169-4924-a666-b75ea4bc2aeb/b0c6e875-56fd-4a79-9737-deb22c9bb7f9"
-					(reference "#PWR037")
-					(unit 1)

Commit message: done
Parts:
- renumbered C17 to C48, C18 to C49, C38 to C50, R23 to R51, R32 to R52, R33 to R53, R34 to R54, U8 to U16
Other:
- added sheet LT3042v3 (lt3042v3.kicad_sch)
Changed lines of the file:
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@@
 		(dnp no)
 		(fields_autoplaced yes)
-		(property "Reference" "R32"
+		(property "Reference" "R52"
 			(at 171.45 100.3299 0)
 			(show_name no)
@@
 		(instances
 			(project "DAC11001"
+				(path "/688e2b68-3871-489b-b27a-c18d3c11fcf6/9763c458-ad2a-49f6-b267-7cfd74c6fed3"
+					(reference "R40")
+					(unit 1)
+				)
+			)
+			(project "DAC11001"
 				(path "/abdba638-bc95-4869-83fe-bbcdf8030f26"
 					(reference "R32")
+					(unit 1)
+				)
+			)
+			(project "DAC11001"
+				(path "/d47dddaa-1169-4924-a666-b75ea4bc2aeb/a8da5177-43c4-4665-b682-d49b9fc3d5b2/9763c458-ad2a-49f6-b267-7cfd74c6fed3"
+					(reference "R52")
 					(unit 1)
 				)
@@
 		(dnp no)
 		(fields_autoplaced yes)
-		(property "Reference" "C17"
+		(property "Reference" "C48"
 			(at 74.93 80.0099 0)
 			(show_name no)
@@
 		(instances
 			(project "DAC11001"
+				(path "/688e2b68-3871-489b-b27a-c18d3c11fcf6/9763c458-ad2a-49f6-b267-7cfd74c6fed3"
+					(reference "C37")
+					(unit 1)
+				)
+			)
+			(project "DAC11001"
 				(path "/abdba638-bc95-4869-83fe-bbcdf8030f26"
 					(reference "C17")
+					(unit 1)
+				)
+			)
+			(project "DAC11001"
+				(path "/d47dddaa-1169-4924-a666-b75ea4bc2aeb/a8da5177-43c4-4665-b682-d49b9fc3d5b2/9763c458-ad2a-49f6-b267-7cfd74c6fed3"
+					(reference "C48")
 					(unit 1)
 				)
@@
 		(dnp no)
 		(fields_autoplaced yes)
-		(property "Reference" "R23"
+		(property "Reference" "R51"
 			(at 100.33 101.5999 0)
 			(show_name no)
@@
 		(instances
 			(project "DAC11001"
+				(path "/688e2b68-3871-489b-b27a-c18d3c11fcf6/9763c458-ad2a-49f6-b267-7cfd74c6fed3"
+					(reference "R39")
+					(unit 1)
+				)
+			)
+			(project "DAC11001"
 				(path "/abdba638-bc95-4869-83fe-bbcdf8030f26"
 					(reference "R23")
+					(unit 1)
+				)
+			)
+			(project "DAC11001"
+				(path "/d47dddaa-1169-4924-a666-b75ea4bc2aeb/a8da5177-43c4-4665-b682-d49b9fc3d5b2/9763c458-ad2a-49f6-b267-7cfd74c6fed3"
+					(reference "R51")
 					(unit 1)
 				)
@@
 		(dnp no)
 		(fields_autoplaced yes)
-		(property "Reference" "U8"
+		(property "Reference" "U16"
 			(at 128.27 67.31 0)
 			(show_name no)
@@
 		(instances
 			(project "DAC11001"
+				(path "/688e2b68-3871-489b-b27a-c18d3c11fcf6/9763c458-ad2a-49f6-b267-7cfd74c6fed3"
+					(reference "U6")
+					(unit 1)
+				)
+			)
+			(project "DAC11001"
 				(path "/abdba638-bc95-4869-83fe-bbcdf8030f26"
 					(reference "U8")
+					(unit 1)
+				)
+			)
+			(project "DAC11001"
+				(path "/d47dddaa-1169-4924-a666-b75ea4bc2aeb/a8da5177-43c4-4665-b682-d49b9fc3d5b2/9763c458-ad2a-49f6-b267-7cfd74c6fed3"
+					(reference "U16")
 					(unit 1)
 				)
@@
 		(dnp no)
 		(fields_autoplaced yes)
-		(property "Reference" "R34"
+		(property "Reference" "R54"
 			(at 195.58 95.2499 0)
 			(show_name no)
@@
 		(instances
 			(project "DAC11001"
+				(path "/688e2b68-3871-489b-b27a-c18d3c11fcf6/9763c458-ad2a-49f6-b267-7cfd74c6fed3"
+					(reference "R42")
+					(unit 1)
+				)
+			)
+			(project "DAC11001"
 				(path "/abdba638-bc95-4869-83fe-bbcdf8030f26"
 					(reference "R34")
+					(unit 1)
+				)
+			)
+			(project "DAC11001"
+				(path "/d47dddaa-1169-4924-a666-b75ea4bc2aeb/a8da5177-43c4-4665-b682-d49b9fc3d5b2/9763c458-ad2a-49f6-b267-7cfd74c6fed3"
+					(reference "R54")
 					(unit 1)
 				)
@@
 		(dnp no)
 		(fields_autoplaced yes)
-		(property "Reference" "C38"
+		(property "Reference" "C50"
 			(at 212.09 92.7099 0)
 			(show_name no)
@@
 		(instances
 			(project "DAC11001"
+				(path "/688e2b68-3871-489b-b27a-c18d3c11fcf6/9763c458-ad2a-49f6-b267-7cfd74c6fed3"
+					(reference "C41")
+					(unit 1)
+				)
+			)
+			(project "DAC11001"
 				(path "/abdba638-bc95-4869-83fe-bbcdf8030f26"
 					(reference "C38")
+					(unit 1)
+				)
+			)
+			(project "DAC11001"
+				(path "/d47dddaa-1169-4924-a666-b75ea4bc2aeb/a8da5177-43c4-4665-b682-d49b9fc3d5b2/9763c458-ad2a-49f6-b267-7cfd74c6fed3"
+					(reference "C50")
 					(unit 1)
 				)
@@
 		(dnp no)
 		(fields_autoplaced yes)
-		(property "Reference" "C18"
+		(property "Reference" "C49"
 			(at 163.83 100.3299 0)
 			(show_name no)
@@
 		(instances
 			(project "DAC11001"
+				(path "/688e2b68-3871-489b-b27a-c18d3c11fcf6/9763c458-ad2a-49f6-b267-7cfd74c6fed3"
+					(reference "C40")
+					(unit 1)
+				)
+			)
+			(project "DAC11001"
 				(path "/abdba638-bc95-4869-83fe-bbcdf8030f26"
 					(reference "C18")
+					(unit 1)
+				)
+			)
+			(project "DAC11001"
+				(path "/d47dddaa-1169-4924-a666-b75ea4bc2aeb/a8da5177-43c4-4665-b682-d49b9fc3d5b2/9763c458-ad2a-49f6-b267-7cfd74c6fed3"
+					(reference "C49")
 					(unit 1)
 				)
@@
 		(dnp no)
 		(fields_autoplaced yes)
-		(property "Reference" "R33"
+		(property "Reference" "R53"
 			(at 195.58 85.0899 0)
 			(show_name no)
@@
 		(instances
 			(project "DAC11001"
+				(path "/688e2b68-3871-489b-b27a-c18d3c11fcf6/9763c458-ad2a-49f6-b267-7cfd74c6fed3"
+					(reference "R41")
+					(unit 1)
+				)
+			)
+			(project "DAC11001"
 				(path "/abdba638-bc95-4869-83fe-bbcdf8030f26"
 					(reference "R33")
+					(unit 1)
+				)
+			)
+			(project "DAC11001"
+				(path "/d47dddaa-1169-4924-a666-b75ea4bc2aeb/a8da5177-43c4-4665-b682-d49b9fc3d5b2/9763c458-ad2a-49f6-b267-7cfd74c6fed3"
+					(reference "R53")
 					(unit 1)
 				)
@@
 		(instances
 			(project "DAC11001"
+				(path "/688e2b68-3871-489b-b27a-c18d3c11fcf6/9763c458-ad2a-49f6-b267-7cfd74c6fed3"
+					(reference "#PWR037")
+					(unit 1)
+				)
+			)
+			(project "DAC11001"
 				(path "/abdba638-bc95-4869-83fe-bbcdf8030f26"
 					(reference "#PWR037")
@@
 				)
 			)
+			(project "DAC11001"
+				(path "/d47dddaa-1169-4924-a666-b75ea4bc2aeb/a8da5177-43c4-4665-b682-d49b9fc3d5b2/9763c458-ad2a-49f6-b267-7cfd74c6fed3"
+					(reference "#PWR037")
+					(unit 1)
+				)
+			)
+		)
+	)
+	(sheet
+		(at 64.77 158.75)
+		(size 31.75 11.43)
+		(exclude_from_sim no)
+		(in_bom yes)
+		(on_board yes)
+		(dnp no)
+		(fields_autoplaced yes)
+		(stroke
+			(width 0.1524)
+			(type solid)
+		)
+		(fill
+			(color 0 0 0 0)
+		)
+		(property "Sheetname" "LT3042v3"
+			(at 64.77 158.0384 0)
+			(show_name no)
+			(do_not_autoplace no)
+			(effects
+				(font
+					(size 1.27 1.27)
+				)
+				(justify left bottom)
+			)
+		)
+		(property "Sheetfile" "lt3042v3.kicad_sch"
+			(at 64.77 170.7646 0)
+			(show_name no)
+			(do_not_autoplace no)
+			(effects
+				(font
+					(size 1.27 1.27)
+				)
+				(justify left top)
+			)
+		)
+		(instances
+			(project ""
+				(path "/688e2b68-3871-489b-b27a-c18d3c11fcf6/9763c458-ad2a-49f6-b267-7cfd74c6fed3"
+					(page "5")
+				)
+			)
+			(project ""
+				(path "/a8da5177-43c4-4665-b682-d49b9fc3d5b2/9763c458-ad2a-49f6-b267-7cfd74c6fed3"
+					(page "")
+				)
+			)
+			(project "DAC11001"
+				(path "/d47dddaa-1169-4924-a666-b75ea4bc2aeb/a8da5177-43c4-4665-b682-d49b9fc3d5b2/9763c458-ad2a-49f6-b267-7cfd74c6fed3"
+					(page "6")
+				)
+			)
