File: lt3094.kicad_sch (KiCad schematic)
At the start: 8 parts, among them U4 LT3094MPDD-PBF

Commit message: main
Changed lines of the file:
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@@
-		)
-	)
-	(label "V_OUT_-16.5"
-		(at 72.39 68.58 0)
-		(effects
-			(font
-				(size 1.27 1.27)
-			)
-			(justify left bottom)
 		)
 	)
@@
 		)
 	)
+	(hierarchical_label "V_OUT_-16.5"
+		(shape input)
+		(at 72.39 68.58 180)
+		(effects
+			(font
+				(size 1.27 1.27)
+			)
+			(justify right)
+		)
+	)

Commit message: main
Connections:
- net V_C_-15 renamed V_C_-15V
Changed lines of the file:
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@@
-		)
-	)
-	(label "V_C_-15"
-		(at 237.49 74.93 0)
-		(effects
-			(font
-				(size 1.27 1.27)
-			)
-			(justify left bottom)
 		)
 	)
@@
 			)
 			(justify right)
+		)
+	)
+	(hierarchical_label "V_C_-15V"
+		(shape input)
+		(at 237.49 74.93 0)
+		(effects
+			(font
+				(size 1.27 1.27)
+			)
+			(justify left)
 		)
 	)
@@
 		(instances
 			(project "DAC11001"
-				(path "/d47dddaa-1169-4924-a666-b75ea4bc2aeb/5ad28e6f-ee73-4b65-bae6-2cd262b8ea89/674a7779-f709-41a4-ab06-7cf143a54cee/e391d005-bed1-43eb-828e-6526cc758b63"
+				(path "/d47dddaa-1169-4924-a666-b75ea4bc2aeb/4741fee4-9c57-455d-b057-ec5a23de6781"
+					(reference "C39")
+					(unit 1)
+				)
+			)
+			(project "DAC11001"
+				(path "/e0aa5e38-0527-4cf2-b522-8958e99675c0/99355de9-7e09-497d-8267-eff07b009003"
 					(reference "C7")
 					(unit 1)
@@
 		(instances
 			(project "DAC11001"
-				(path "/d47dddaa-1169-4924-a666-b75ea4bc2aeb/5ad28e6f-ee73-4b65-bae6-2cd262b8ea89/674a7779-f709-41a4-ab06-7cf143a54cee/e391d005-bed1-43eb-828e-6526cc758b63"
+				(path "/d47dddaa-1169-4924-a666-b75ea4bc2aeb/4741fee4-9c57-455d-b057-ec5a23de6781"
+					(reference "C40")
+					(unit 1)
+				)
+			)
+			(project "DAC11001"
+				(path "/e0aa5e38-0527-4cf2-b522-8958e99675c0/99355de9-7e09-497d-8267-eff07b009003"
 					(reference "C8")
 					(unit 1)
@@
 		(instances
 			(project "DAC11001"
-				(path "/d47dddaa-1169-4924-a666-b75ea4bc2aeb/5ad28e6f-ee73-4b65-bae6-2cd262b8ea89/674a7779-f709-41a4-ab06-7cf143a54cee/e391d005-bed1-43eb-828e-6526cc758b63"
+				(path "/d47dddaa-1169-4924-a666-b75ea4bc2aeb/4741fee4-9c57-455d-b057-ec5a23de6781"
+					(reference "R36")
+					(unit 1)
+				)
+			)
+			(project "DAC11001"
+				(path "/e0aa5e38-0527-4cf2-b522-8958e99675c0/99355de9-7e09-497d-8267-eff07b009003"
 					(reference "R9")
 					(unit 1)
@@
 		(instances
 			(project "DAC11001"
-				(path "/d47dddaa-1169-4924-a666-b75ea4bc2aeb/5ad28e6f-ee73-4b65-bae6-2cd262b8ea89/674a7779-f709-41a4-ab06-7cf143a54cee/e391d005-bed1-43eb-828e-6526cc758b63"
+				(path "/d47dddaa-1169-4924-a666-b75ea4bc2aeb/4741fee4-9c57-455d-b057-ec5a23de6781"
+					(reference "R37")
+					(unit 1)
+				)
+			)
+			(project "DAC11001"
+				(path "/e0aa5e38-0527-4cf2-b522-8958e99675c0/99355de9-7e09-497d-8267-eff07b009003"
 					(reference "R10")
 					(unit 1)
@@
 		(instances
 			(project "DAC11001"
-				(path "/d47dddaa-1169-4924-a666-b75ea4bc2aeb/5ad28e6f-ee73-4b65-bae6-2cd262b8ea89/674a7779-f709-41a4-ab06-7cf143a54cee/e391d005-bed1-43eb-828e-6526cc758b63"
+				(path "/d47dddaa-1169-4924-a666-b75ea4bc2aeb/4741fee4-9c57-455d-b057-ec5a23de6781"
+					(reference "C41")
+					(unit 1)
+				)
+			)
+			(project "DAC11001"
+				(path "/e0aa5e38-0527-4cf2-b522-8958e99675c0/99355de9-7e09-497d-8267-eff07b009003"
 					(reference "C9")
 					(unit 1)
@@
 		(instances
 			(project "DAC11001"
-				(path "/d47dddaa-1169-4924-a666-b75ea4bc2aeb/5ad28e6f-ee73-4b65-bae6-2cd262b8ea89/674a7779-f709-41a4-ab06-7cf143a54cee/e391d005-bed1-43eb-828e-6526cc758b63"
+				(path "/d47dddaa-1169-4924-a666-b75ea4bc2aeb/4741fee4-9c57-455d-b057-ec5a23de6781"
+					(reference "R38")
+					(unit 1)
+				)
+			)
+			(project "DAC11001"
+				(path "/e0aa5e38-0527-4cf2-b522-8958e99675c0/99355de9-7e09-497d-8267-eff07b009003"
 					(reference "R11")
 					(unit 1)
@@
 		(instances
 			(project "DAC11001"
-				(path "/d47dddaa-1169-4924-a666-b75ea4bc2aeb/5ad28e6f-ee73-4b65-bae6-2cd262b8ea89/674a7779-f709-41a4-ab06-7cf143a54cee/e391d005-bed1-43eb-828e-6526cc758b63"
+				(path "/d47dddaa-1169-4924-a666-b75ea4bc2aeb/4741fee4-9c57-455d-b057-ec5a23de6781"
+					(reference "U10")
+					(unit 1)
+				)
+			)
+			(project "DAC11001"
+				(path "/e0aa5e38-0527-4cf2-b522-8958e99675c0/99355de9-7e09-497d-8267-eff07b009003"
 					(reference "U4")
 					(unit 1)
@@
 		(dnp no)
 		(fields_autoplaced yes)
-		(property "Reference" "#PWR020"
+		(property "Reference" "#PWR021"
 			(at 113.03 107.95 0)
 			(hide yes)
@@
 		(instances
 			(project "DAC11001"
-				(path "/d47dddaa-1169-4924-a666-b75ea4bc2aeb/5ad28e6f-ee73-4b65-bae6-2cd262b8ea89/674a7779-f709-41a4-ab06-7cf143a54cee/e391d005-bed1-43eb-828e-6526cc758b63"
+				(path "/d47dddaa-1169-4924-a666-b75ea4bc2aeb/4741fee4-9c57-455d-b057-ec5a23de6781"
 					(reference "#PWR020")
+					(unit 1)
+				)
+			)
+			(project "DAC11001"
+				(path "/e0aa5e38-0527-4cf2-b522-8958e99675c0/99355de9-7e09-497d-8267-eff07b009003"
+					(reference "#PWR021")
 					(unit 1)
 				)
@@
 		(instances
 			(project "DAC11001"
-				(path "/d47dddaa-1169-4924-a666-b75ea4bc2aeb/5ad28e6f-ee73-4b65-bae6-2cd262b8ea89/674a7779-f709-41a4-ab06-7cf143a54cee/e391d005-bed1-43eb-828e-6526cc758b63"
+				(path "/d47dddaa-1169-4924-a666-b75ea4bc2aeb/4741fee4-9c57-455d-b057-ec5a23de6781"
+					(reference "R35")
+					(unit 1)
+				)
+			)
+			(project "DAC11001"
+				(path "/e0aa5e38-0527-4cf2-b522-8958e99675c0/99355de9-7e09-497d-8267-eff07b009003"
 					(reference "R8")
 					(unit 1)

Commit message: modular
Connections:
- net V_C_-15V renamed V_P_C_-15V
- net V_OUT_-16.5 renamed V_P_-16.5V
