File: lt3094.kicad_sch (KiCad schematic)
At the start: 8 parts, among them U4 LT3094MPDD-PBF

Commit message: globaled
Changed lines of the file:
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@@
+	)
+	(junction
+		(at 209.55 80.01)
+		(diameter 0)
+		(color 0 0 0 0)
 	)
 	(junction
@@
 		(color 0 0 0 0)
 	)
-	(junction
-		(at 209.55 80.01)
-		(diameter 0)
-		(color 0 0 0 0)
-	)
 	(wire
 		(pts
@@
 	(wire
 		(pts
-			(xy 209.55 80.01) (xy 228.6 80.01)
+			(xy 209.55 71.12) (xy 237.49 71.12)
 		)
 		(stroke
@@
 	(wire
 		(pts
+			(xy 209.55 71.12) (xy 209.55 80.01)
+		)
+		(stroke
+			(width 0)
+			(type default)
+		)
+	)
+	(wire
+		(pts
 			(xy 209.55 80.01) (xy 209.55 90.17)
 		)
@@
 		)
 	)
-	(label "V_P_C_-15V"
-		(at 228.6 80.01 0)
+	(global_label "V_P_-16.5V"
+		(shape input)
+		(at 63.5 73.66 180)
+		(fields_autoplaced yes)
 		(effects
 			(font
 				(size 1.27 1.27)
 			)
-			(justify left bottom)
-		)
-	)
-	(label "V_P_-16.5V"
-		(at 63.5 73.66 0)
+			(justify right)
+		)
+		(property "Intersheetrefs" "${INTERSHEET_REFS}"
+			(at 49.3267 73.66 0)
+			(hide yes)
+			(show_name no)
+			(do_not_autoplace no)
+			(effects
+				(font
+					(size 1.27 1.27)
+				)
+				(justify right)
+			)
+		)
+	)
+	(global_label "V_P_C_-15V"
+		(shape input)
+		(at 237.49 71.12 0)
+		(fields_autoplaced yes)
 		(effects
 			(font
 				(size 1.27 1.27)
 			)
-			(justify left bottom)
+			(justify left)
+		)
+		(property "Intersheetrefs" "${INTERSHEET_REFS}"
+			(at 252.0866 71.12 0)
+			(hide yes)
+			(show_name no)
+			(do_not_autoplace no)
+			(effects
+				(font
+					(size 1.27 1.27)
+				)
+				(justify left)
+			)
 		)
 	)
@@
 				)
 			)
-			(project "DAC11001"
-				(path "/d47dddaa-1169-4924-a666-b75ea4bc2aeb/2354dc51-baac-49c4-b0f2-6409abc4ef9d"
-					(reference "R49")
-					(unit 1)
-				)
-			)
 		)
 	)
@@
 				)
 			)
-			(project "DAC11001"
-				(path "/d47dddaa-1169-4924-a666-b75ea4bc2aeb/2354dc51-baac-49c4-b0f2-6409abc4ef9d"
-					(reference "R50")
-					(unit 1)
-				)
-			)
 		)
 	)
@@
 				)
 			)
-			(project "DAC11001"
-				(path "/d47dddaa-1169-4924-a666-b75ea4bc2aeb/2354dc51-baac-49c4-b0f2-6409abc4ef9d"
-					(reference "C45")
-					(unit 1)
-				)
-			)
 		)
 	)
@@
 				)
 			)
-			(project "DAC11001"
-				(path "/d47dddaa-1169-4924-a666-b75ea4bc2aeb/2354dc51-baac-49c4-b0f2-6409abc4ef9d"
-					(reference "#PWR021")
-					(unit 1)
-				)
-			)
 		)
 	)
@@
 				)
 			)
-			(project "DAC11001"
-				(path "/d47dddaa-1169-4924-a666-b75ea4bc2aeb/2354dc51-baac-49c4-b0f2-6409abc4ef9d"
-					(reference "C43")
-					(unit 1)
-				)
-			)
 		)
 	)
@@
 				)
 			)
-			(project "DAC11001"
-				(path "/d47dddaa-1169-4924-a666-b75ea4bc2aeb/2354dc51-baac-49c4-b0f2-6409abc4ef9d"
-					(reference "U15")
-					(unit 1)
-				)
-			)
 		)
 	)
@@
 				)
 			)
-			(project "DAC11001"
-				(path "/d47dddaa-1169-4924-a666-b75ea4bc2aeb/2354dc51-baac-49c4-b0f2-6409abc4ef9d"
-					(reference "R48")
-					(unit 1)
-				)
-			)
 		)
 	)
@@
 				)
 			)
-			(project "DAC11001"
-				(path "/d47dddaa-1169-4924-a666-b75ea4bc2aeb/2354dc51-baac-49c4-b0f2-6409abc4ef9d"
-					(reference "C44")
-					(unit 1)
-				)
-			)
 		)
 	)
@@
 				)
 			)
-			(project "DAC11001"
-				(path "/d47dddaa-1169-4924-a666-b75ea4bc2aeb/2354dc51-baac-49c4-b0f2-6409abc4ef9d"
-					(reference "R47")
-					(unit 1)
-				)
-			)
-		)
-	)
-	(sheet_instances
-		(path "/"
-			(page "6")
-		)
-	)
+		)
+	)
