File: lt3999.kicad_sch (KiCad schematic)
At the start: 20 parts, among them T2 Transformer_SP_2S, U11 LT3999EDD-PBF

Commit message: main
Connections:
- net V_OUT_+16.5 renamed LT3042/V_OUT_+16.5
- net V_OUT_-16.5: no longer names the net of C22.1, L4.2
Other:
- sheet LT3042 ports: added V_OUT_+16.5; removed none
- moved on the sheet: C19, C20, C21, C22, D5, D6, D7, D8, L3, L4, R24, R25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

Commit message: modular
Connections:
- net V_P_-16.5V: now reaches C22.1, L4.2
- net LT3042/V_OUT_+16.5 renamed V_P_+16.5V
- net V_EX_INPUT renamed V_P_EX_INPUT
Other:
- removed sheet LT3042
- removed sheet LT3094
