File: lt3999.kicad_sch (KiCad schematic)
At the start: 20 parts, among them T2 Transformer_SP_2S, U11 LT3999EDD-PBF

Commit message: main
Parts:
- renumbered C19 to C14, C20 to C15, C21 to C16, C22 to C37, D5 to D1, D8 to D10, D6 to D4, D7 to D9, L3 to L1, L4 to L2, R24 to R19, R25 to R20, R26 to R21, R27 to R22, R28 to R39, R29 to R40, R30 to R41, R31 to R42, T2 to T1, U11 to U1
Changed lines of the file:
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@@
 		(dnp no)
 		(fields_autoplaced yes)
-		(property "Reference" "C20"
+		(property "Reference" "C15"
 			(at 153.67 50.7999 0)
 			(show_name no)
@@
 				)
 			)
+			(project "DAC11001"
+				(path "/d47dddaa-1169-4924-a666-b75ea4bc2aeb/d3048a48-51ba-4481-ad89-7603f55b3b15"
+					(reference "C15")
+					(unit 1)
+				)
+			)
 		)
 	)
@@
 		(dnp no)
 		(fields_autoplaced yes)
-		(property "Reference" "L4"
+		(property "Reference" "L2"
 			(at 247.65 58.42 90)
 			(show_name no)
@@
 				)
 			)
+			(project "DAC11001"
+				(path "/d47dddaa-1169-4924-a666-b75ea4bc2aeb/d3048a48-51ba-4481-ad89-7603f55b3b15"
+					(reference "L2")
+					(unit 1)
+				)
+			)
 		)
 	)
@@
 				)
 			)
+			(project "DAC11001"
+				(path "/d47dddaa-1169-4924-a666-b75ea4bc2aeb/d3048a48-51ba-4481-ad89-7603f55b3b15"
+					(reference "#PWR018")
+					(unit 1)
+				)
+			)
 		)
 	)
@@
 		(dnp no)
 		(fields_autoplaced yes)
-		(property "Reference" "R30"
+		(property "Reference" "R41"
 			(at 152.4 58.4199 0)
 			(show_name no)
@@
 				)
 			)
+			(project "DAC11001"
+				(path "/d47dddaa-1169-4924-a666-b75ea4bc2aeb/d3048a48-51ba-4481-ad89-7603f55b3b15"
+					(reference "R41")
+					(unit 1)
+				)
+			)
 		)
 	)
@@
 		(dnp no)
 		(fields_autoplaced yes)
-		(property "Reference" "D6"
+		(property "Reference" "D4"
 			(at 214.63 36.83 0)
 			(show_name no)
@@
 				)
 			)
+			(project "DAC11001"
+				(path "/d47dddaa-1169-4924-a666-b75ea4bc2aeb/d3048a48-51ba-4481-ad89-7603f55b3b15"
+					(reference "D4")
+					(unit 1)
+				)
+			)
 		)
 	)
@@
 		(dnp no)
 		(fields_autoplaced yes)
-		(property "Reference" "D5"
+		(property "Reference" "D1"
 			(at 204.47 40.64 0)
 			(show_name no)
@@
 				)
 			)
+			(project "DAC11001"
+				(path "/d47dddaa-1169-4924-a666-b75ea4bc2aeb/d3048a48-51ba-4481-ad89-7603f55b3b15"
+					(reference "D1")
+					(unit 1)
+				)
+			)
 		)
 	)
@@
 		(dnp no)
 		(fields_autoplaced yes)
-		(property "Reference" "U11"
+		(property "Reference" "U1"
 			(at 101.6 62.23 0)
 			(show_name no)
@@
 				)
 			)
+			(project "DAC11001"
+				(path "/d47dddaa-1169-4924-a666-b75ea4bc2aeb/d3048a48-51ba-4481-ad89-7603f55b3b15"
+					(reference "U1")
+					(unit 1)
+				)
+			)
 		)
 	)
@@
 		(dnp no)
 		(fields_autoplaced yes)
-		(property "Reference" "D8"
+		(property "Reference" "D10"
 			(at 227.33 57.15 0)
 			(show_name no)
@@
 				)
 			)
+			(project "DAC11001"
+				(path "/d47dddaa-1169-4924-a666-b75ea4bc2aeb/d3048a48-51ba-4481-ad89-7603f55b3b15"
+					(reference "D10")
+					(unit 1)
+				)
+			)
 		)
 	)
@@
 		(dnp no)
 		(fields_autoplaced yes)
-		(property "Reference" "R31"
+		(property "Reference" "R42"
 			(at 242.57 52.0699 0)
 			(show_name no)
@@
 				)
 			)
+			(project "DAC11001"
+				(path "/d47dddaa-1169-4924-a666-b75ea4bc2aeb/d3048a48-51ba-4481-ad89-7603f55b3b15"
+					(reference "R42")
+					(unit 1)
+				)
+			)
 		)
 	)
@@
 		(dnp no)
 		(fields_autoplaced yes)
-		(property "Reference" "C21"
+		(property "Reference" "C16"
 			(at 255.27 45.7199 0)
 			(show_name no)
@@
 				)
 			)
+			(project "DAC11001"
+				(path "/d47dddaa-1169-4924-a666-b75ea4bc2aeb/d3048a48-51ba-4481-ad89-7603f55b3b15"
+					(reference "C16")
+					(unit 1)
+				)
+			)
 		)
 	)
@@
 		(dnp no)
 		(fields_autoplaced yes)
-		(property "Reference" "R26"
+		(property "Reference" "R21"
 			(at 46.99 102.8699 0)
 			(show_name no)
@@
 				)
 			)
+			(project "DAC11001"
+				(path "/d47dddaa-1169-4924-a666-b75ea4bc2aeb/d3048a48-51ba-4481-ad89-7603f55b3b15"
+					(reference "R21")
+					(unit 1)
+				)
+			)
 		)
 	)
@@
 		(dnp no)
 		(fields_autoplaced yes)
-		(property "Reference" "D7"
+		(property "Reference" "D9"
 			(at 215.9 52.07 0)
 			(show_name no)
@@
 				)
 			)
+			(project "DAC11001"
+				(path "/d47dddaa-1169-4924-a666-b75ea4bc2aeb/d3048a48-51ba-4481-ad89-7603f55b3b15"
+					(reference "D9")
+					(unit 1)
+				)
+			)
 		)
 	)
@@
 				)
 			)
+			(project "DAC11001"
+				(path "/d47dddaa-1169-4924-a666-b75ea4bc2aeb/d3048a48-51ba-4481-ad89-7603f55b3b15"
+					(reference "#PWR016")
+					(unit 1)
+				)
+			)
 		)
 	)
@@
 				)
 			)
+			(project "DAC11001"
+				(path "/d47dddaa-1169-4924-a666-b75ea4bc2aeb/d3048a48-51ba-4481-ad89-7603f55b3b15"
+					(reference "#PWR015")
+					(unit 1)
+				)
+			)
 		)
 	)
@@
 		(dnp no)
 		(fields_autoplaced yes)
-		(property "Reference" "C19"
+		(property "Reference" "C14"
 			(at 138.43 100.3299 0)
 			(show_name no)
@@
 				)
 			)
+			(project "DAC11001"
+				(path "/d47dddaa-1169-4924-a666-b75ea4bc2aeb/d3048a48-51ba-4481-ad89-7603f55b3b15"
+					(reference "C14")
+					(unit 1)
+				)
+			)
 		)
 	)
@@
 		(dnp no)
 		(fields_autoplaced yes)
-		(property "Reference" "R28"
+		(property "Reference" "R39"
 			(at 120.65 99.0599 0)
 			(show_name no)
@@
 				)
 			)
+			(project "DAC11001"
+				(path "/d47dddaa-1169-4924-a666-b75ea4bc2aeb/d3048a48-51ba-4481-ad89-7603f55b3b15"
+					(reference "R39")
+					(unit 1)
+				)
+			)
 		)
 	)
@@
 		(dnp no)
 		(fields_autoplaced yes)
-		(property "Reference" "L3"
+		(property "Reference" "L1"
 			(at 247.65 38.1 90)
 			(show_name no)
@@
 				)
 			)
+			(project "DAC11001"
+				(path "/d47dddaa-1169-4924-a666-b75ea4bc2aeb/d3048a48-51ba-4481-ad89-7603f55b3b15"
+					(reference "L1")
+					(unit 1)
+				)
+			)
 		)
 	)
@@
 		(dnp no)
 		(fields_autoplaced yes)
-		(property "Reference" "R29"
+		(property "Reference" "R40"
 			(at 128.27 99.0599 0)
 			(show_name no)
@@
 				)
 			)
+			(project "DAC11001"
+				(path "/d47dddaa-1169-4924-a666-b75ea4bc2aeb/d3048a48-51ba-4481-ad89-7603f55b3b15"
+					(reference "R40")
+					(unit 1)
+				)
+			)
 		)
 	)
@@
 		(dnp no)
 		(fields_autoplaced yes)
-		(property "Reference" "R27"
+		(property "Reference" "R22"
 			(at 71.12 97.7899 0)
 			(show_name no)
@@
 				)
 			)
+			(project "DAC11001"
+				(path "/d47dddaa-1169-4924-a666-b75ea4bc2aeb/d3048a48-51ba-4481-ad89-7603f55b3b15"
+					(reference "R22")
+					(unit 1)
+				)
+			)
 		)
 	)
@@
 		(dnp no)
 		(fields_autoplaced yes)
-		(property "Reference" "C22"
+		(property "Reference" "C37"
 			(at 255.27 66.0399 0)
 			(show_name no)
@@
 				)
 			)
+			(project "DAC11001"
+				(path "/d47dddaa-1169-4924-a666-b75ea4bc2aeb/d3048a48-51ba-4481-ad89-7603f55b3b15"
+					(reference "C37")
+					(unit 1)
+				)
+			)
 		)
 	)
@@
 		(dnp no)
 		(fields_autoplaced yes)
-		(property "Reference" "T2"
+		(property "Reference" "T1"
 			(at 181.61 38.1 0)
 			(show_name no)
@@
 				)
 			)
+			(project "DAC11001"
+				(path "/d47dddaa-1169-4924-a666-b75ea4bc2aeb/d3048a48-51ba-4481-ad89-7603f55b3b15"
+					(reference "T1")
+					(unit 1)
+				)
+			)
 		)
 	)
@@
 		(dnp no)
 		(fields_autoplaced yes)
-		(property "Reference" "R25"
+		(property "Reference" "R20"
 			(at 46.99 92.7099 0)
 			(show_name no)
@@
 				)
 			)
+			(project "DAC11001"
+				(path "/d47dddaa-1169-4924-a666-b75ea4bc2aeb/d3048a48-51ba-4481-ad89-7603f55b3b15"
+					(reference "R20")
+					(unit 1)
+				)
+			)
 		)
 	)
@@
 				)
 			)
+			(project "DAC11001"
+				(path "/d47dddaa-1169-4924-a666-b75ea4bc2aeb/d3048a48-51ba-4481-ad89-7603f55b3b15"
+					(reference "#PWR017")
+					(unit 1)
+				)
+			)
 		)
 	)
@@
 		(dnp no)
 		(fields_autoplaced yes)
-		(property "Reference" "R24"
+		(property "Reference" "R19"
 			(at 46.99 82.5499 0)
 			(show_name no)
@@
 				)
 			)
-		)
-	)
-	(sheet_instances
-		(path "/"
-			(page "11")
-		)
-	)
+			(project "DAC11001"
+				(path "/d47dddaa-1169-4924-a666-b75ea4bc2aeb/d3048a48-51ba-4481-ad89-7603f55b3b15"
+					(reference "R19")
+					(unit 1)
+				)
+			)
+		)
+	)

Commit message: globaled
Parts:
- renumbered C14 to C19, C15 to C20, C16 to C21, C37 to C22, D1 to D5, D4 to D6, D9 to D7, D10 to D8, L1 to L3, L2 to L4, R19 to R24, R20 to R25, R21 to R26, R22 to R27, R39 to R28, R40 to R29, R41 to R30, R42 to R31, T1 to T2, U1 to U11

Commit message: done
Parts:
- renumbered C19 to C52, C20 to C53, C21 to C56, C22 to C57, D5 to D1, D8 to D10, D6 to D4, D7 to D9, L3 to L1, L4 to L2, R24 to R55, R25 to R56, R26 to R57, R27 to R58, R28 to R60, R29 to R61, R30 to R62, R31 to R66, T2 to T1, U11 to U17
Other:
- added sheet LT3042 (lt3042.kicad_sch)
- added sheet LT3042v2 (lt3042v2.kicad_sch)
- added sheet LT3094 (untitled.kicad_sch)
