File: ltc6655ln-5.kicad_sch (KiCad schematic)
At the start: 2 parts, among them U5 LTC6655LNCHMS8-5-PBF

Commit message: modular
Connections:
- net V_12V renamed V_P_+12V
Other:
- removed sheet OPA828_4X
