File: ltc6655ln-5.kicad_sch (KiCad schematic)
At the start: 2 parts, among them U5 LTC6655LNCHMS8-5-PBF

Commit message: globaled
Changed lines of the file:
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@@
 		)
 	)
-	(label "V_P_+12V"
-		(at 82.55 71.12 0)
+	(global_label "V_P_+12V"
+		(shape input)
+		(at 82.55 71.12 180)
+		(fields_autoplaced yes)
 		(effects
 			(font
 				(size 1.27 1.27)
 			)
-			(justify left bottom)
+			(justify right)
+		)
+		(property "Intersheetrefs" "${INTERSHEET_REFS}"
+			(at 70.191 71.12 0)
+			(hide yes)
+			(show_name no)
+			(do_not_autoplace no)
+			(effects
+				(font
+					(size 1.27 1.27)
+				)
+				(justify right)
+			)
 		)
 	)
@@
 		)
 	)
+	(embedded_fonts no)
 )
