File: opa828_4x.kicad_sch (KiCad schematic)
At the start: 27 parts, among them U12 OPA828ID, U13 OPA828ID, U14 OPA828ID, U2 OPA828ID

Commit message: modular
Connections:
- net V_LN_5 renamed LTC6655LN-5/V_LN_5
- net V_N_REF_FORCE renamed V_REF-_FORCE
- net V_N_REF_SENSE renamed V_REF-_SENSE
- net V_P_REF_FORCE renamed V_REF+_FORCE
- net V_P_REF_SENSE renamed V_REF+_SENSE
Other:
- added sheet LTC6655LN-5 (ltc6655ln-5.kicad_sch)
