File: opa828_4x.kicad_sch (KiCad schematic)
At the start: 27 parts, among them U12 OPA828ID, U13 OPA828ID, U14 OPA828ID, U2 OPA828ID

Commit message: main
Connections:
- net V_C_+15V renamed V_P_C_+15V
- net V_C_-15 renamed V_P_C_-15V
Changed lines of the file:
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@@
-	(wire
-		(pts
-			(xy 129.54 35.56) (xy 129.54 48.26)
-		)
-		(stroke
-			(width 0)
-			(type default)
-		)
-	)
 	(wire
 		(pts
@@
 	(wire
 		(pts
+			(xy 129.54 30.48) (xy 129.54 48.26)
+		)
+		(stroke
+			(width 0)
+			(type default)
+		)
+	)
+	(wire
+		(pts
 			(xy 149.86 24.13) (xy 149.86 62.23)
 		)
@@
 		)
 	)
-	(label "V_C_-15"
+	(label "V_P_C_-15V"
+		(at 82.55 90.17 0)
+		(effects
+			(font
+				(size 1.27 1.27)
+			)
+			(justify left bottom)
+		)
+	)
+	(label "V_P_C_+15V"
+		(at 229.87 110.49 0)
+		(effects
+			(font
+				(size 1.27 1.27)
+			)
+			(justify left bottom)
+		)
+	)
+	(label "V_P_C_+15V"
+		(at 229.87 38.1 0)
+		(effects
+			(font
+				(size 1.27 1.27)
+			)
+			(justify left bottom)
+		)
+	)
+	(label "V_P_C_-15V"
+		(at 182.88 90.17 0)
+		(effects
+			(font
+				(size 1.27 1.27)
+			)
+			(justify left bottom)
+		)
+	)
+	(label "V_P_C_+15V"
+		(at 129.54 30.48 0)
+		(effects
+			(font
+				(size 1.27 1.27)
+			)
+			(justify left bottom)
+		)
+	)
+	(label "V_P_C_-15V"
 		(at 184.15 166.37 0)
 		(effects
@@
 		)
 	)
-	(label "V_C_-15"
-		(at 182.88 90.17 0)
-		(effects
-			(font
-				(size 1.27 1.27)
-			)
-			(justify left bottom)
-		)
-	)
-	(label "V_C_-15"
-		(at 82.55 90.17 0)
-		(effects
-			(font
-				(size 1.27 1.27)
-			)
-			(justify left bottom)
-		)
-	)
-	(label "V_C_-15"
+	(label "V_P_C_+15V"
+		(at 154.94 114.3 0)
+		(effects
+			(font
+				(size 1.27 1.27)
+			)
+			(justify left bottom)
+		)
+	)
+	(label "V_P_C_-15V"
 		(at 100.33 167.64 0)
 		(effects
 			(font
-				(size 1.27 1.27)
-			)
-			(justify left bottom)
-		)
-	)
-	(label "V_C_+15V"
-		(at 229.87 38.1 0)
-		(effects
-			(font
-				(size 1.27 1.27)
-			)
-			(justify left bottom)
-		)
-	)
-	(label "V_C_+15V"
-		(at 229.87 110.49 0)
-		(effects
-			(font
-				(size 1.27 1.27)
-			)
-			(justify left bottom)
-		)
-	)
-	(label "V_C_+15V"
-		(at 154.94 114.3 0)
-		(effects
-			(font
-				(size 1.27 1.27)
-			)
-			(justify left bottom)
-		)
-	)
-	(label "V_C_+15V"
-		(at 129.54 35.56 0)
-		(effects
-			(font

Commit message: globaled
Other:
- moved on the sheet: C25
Changed lines of the file:
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@@
 	)
 	(junction
-		(at 184.15 157.48)
+		(at 184.15 153.67)
+		(diameter 0)
+		(color 0 0 0 0)
+	)
+	(junction
+		(at 182.88 81.28)
 		(diameter 0)
 		(color 0 0 0 0)
@@
 		(color 0 0 0 0)
 	)
-	(junction
-		(at 182.88 81.28)
-		(diameter 0)
-		(color 0 0 0 0)
-	)
 	(wire
 		(pts
@@
 	(wire
 		(pts
-			(xy 182.88 81.28) (xy 182.88 90.17)
+			(xy 182.88 81.28) (xy 182.88 91.44)
 		)
 		(stroke
@@
 	(wire
 		(pts
-			(xy 200.66 157.48) (xy 194.31 157.48)
+			(xy 200.66 153.67) (xy 194.31 153.67)
 		)
 		(stroke
@@
 	(wire
 		(pts
-			(xy 184.15 140.97) (xy 184.15 157.48)
+			(xy 184.15 140.97) (xy 184.15 153.67)
 		)
 		(stroke
@@
 	(wire
 		(pts
-			(xy 184.15 157.48) (xy 184.15 166.37)
+			(xy 184.15 153.67) (xy 184.15 162.56)
 		)
 		(stroke
@@
 	(wire
 		(pts
-			(xy 184.15 157.48) (xy 186.69 157.48)
+			(xy 184.15 153.67) (xy 186.69 153.67)
 		)
 		(stroke
@@
 		)
 	)
-	(label "V_P_C_-15V"
-		(at 82.55 90.17 0)
+	(global_label "V_P_C_+15V"
+		(shape input)
+		(at 154.94 114.3 180)
+		(fields_autoplaced yes)
 		(effects
 			(font
 				(size 1.27 1.27)
 			)
-			(justify left bottom)
+			(justify right)
+		)
+		(property "Intersheetrefs" "${INTERSHEET_REFS}"
+			(at 140.3434 114.3 0)
+			(hide yes)
+			(show_name no)
+			(do_not_autoplace no)
+			(effects
+				(font
+					(size 1.27 1.27)
+				)
+				(justify right)
+			)
 		)
 	)
-	(label "V_P_C_+15V"
-		(at 229.87 110.49 0)
+	(global_label "V_P_C_+15V"
+		(shape input)
+		(at 129.54 30.48 180)
+		(fields_autoplaced yes)
 		(effects
 			(font
 				(size 1.27 1.27)
 			)
-			(justify left bottom)
+			(justify right)
+		)
+		(property "Intersheetrefs" "${INTERSHEET_REFS}"
+			(at 114.9434 30.48 0)
+			(hide yes)
+			(show_name no)
+			(do_not_autoplace no)
+			(effects
+				(font
+					(size 1.27 1.27)
+				)
+				(justify right)
+			)
 		)
 	)
-	(label "V_P_C_+15V"
-		(at 229.87 38.1 0)
+	(global_label "V_P_C_+15V"
+		(shape input)
+		(at 229.87 38.1 180)
+		(fields_autoplaced yes)
 		(effects
 			(font
 				(size 1.27 1.27)
 			)
-			(justify left bottom)
+			(justify right)
+		)
+		(property "Intersheetrefs" "${INTERSHEET_REFS}"
+			(at 215.2734 38.1 0)
+			(hide yes)
+			(show_name no)
+			(do_not_autoplace no)
+			(effects
+				(font
+					(size 1.27 1.27)
+				)
+				(justify right)
+			)
 		)
 	)
-	(label "V_P_C_-15V"
-		(at 182.88 90.17 0)
+	(global_label "V_P_C_-15V"
+		(shape input)
+		(at 82.55 90.17 180)
+		(fields_autoplaced yes)
 		(effects
 			(font
 				(size 1.27 1.27)
 			)
-			(justify left bottom)
+			(justify right)
+		)
+		(property "Intersheetrefs" "${INTERSHEET_REFS}"
+			(at 67.9534 90.17 0)
+			(hide yes)
+			(show_name no)
+			(do_not_autoplace no)
+			(effects
+				(font
+					(size 1.27 1.27)
+				)
+				(justify right)
+			)
 		)
 	)
-	(label "V_P_C_+15V"
-		(at 129.54 30.48 0)
+	(global_label "V_P_C_+15V"
+		(shape input)
+		(at 229.87 110.49 180)
+		(fields_autoplaced yes)
 		(effects
 			(font
 				(size 1.27 1.27)
 			)
-			(justify left bottom)
+			(justify right)
+		)
+		(property "Intersheetrefs" "${INTERSHEET_REFS}"
+			(at 215.2734 110.49 0)
+			(hide yes)
+			(show_name no)
+			(do_not_autoplace no)
+			(effects
+				(font
+					(size 1.27 1.27)
+				)
+				(justify right)
+			)
 		)
 	)
-	(label "V_P_C_-15V"
-		(at 184.15 166.37 0)
+	(global_label "V_P_C_-15V"
+		(shape input)
+		(at 184.15 162.56 180)
+		(fields_autoplaced yes)
 		(effects
 			(font
 				(size 1.27 1.27)
 			)
-			(justify left bottom)
+			(justify right)
+		)
+		(property "Intersheetrefs" "${INTERSHEET_REFS}"
+			(at 169.5534 162.56 0)
+			(hide yes)
+			(show_name no)
+			(do_not_autoplace no)
+			(effects
+				(font
+					(size 1.27 1.27)
+				)
+				(justify right)
+			)
 		)
 	)
-	(label "V_P_C_+15V"
-		(at 154.94 114.3 0)
+	(global_label "V_P_C_-15V"
+		(shape input)
+		(at 100.33 167.64 180)
+		(fields_autoplaced yes)
 		(effects
 			(font
 				(size 1.27 1.27)
 			)
-			(justify left bottom)
+			(justify right)
+		)
+		(property "Intersheetrefs" "${INTERSHEET_REFS}"
+			(at 85.7334 167.64 0)
+			(hide yes)
+			(show_name no)
+			(do_not_autoplace no)
+			(effects
+				(font
+					(size 1.27 1.27)
+				)
+				(justify right)
+			)
 		)
 	)
-	(label "V_P_C_-15V"
-		(at 100.33 167.64 0)
+	(global_label "V_P_C_-15V"
+		(shape input)
+		(at 182.88 91.44 180)
+		(fields_autoplaced yes)
 		(effects
 			(font
 				(size 1.27 1.27)
 			)
-			(justify left bottom)
+			(justify right)
+		)
+		(property "Intersheetrefs" "${INTERSHEET_REFS}"
+			(at 168.2834 91.44 0)
+			(hide yes)
+			(show_name no)
+			(do_not_autoplace no)
+			(effects
+				(font
+					(size 1.27 1.27)
+				)
+				(justify right)
+			)
 		)
 	)
@@
 	(symbol
 		(lib_id "power:GNDA")
-		(at 200.66 157.48 0)
+		(at 200.66 153.67 0)
 		(unit 1)
 		(body_style 1)
@@
 		(fields_autoplaced yes)
 		(property "Reference" "#PWR026"
-			(at 200.66 163.83 0)
+			(at 200.66 160.02 0)
 			(hide yes)
 			(show_name no)
@@
 		)
 		(property "Value" "GNDA"
-			(at 200.66 162.56 0)
+			(at 200.66 158.75 0)
 			(show_name no)
 			(do_not_autoplace no)
@@
 		)
 		(property "Footprint" ""
-			(at 200.66 157.48 0)
+			(at 200.66 153.67 0)
 			(hide yes)
 			(show_name no)
@@
 		)
 		(property "Datasheet" ""
-			(at 200.66 157.48 0)
+			(at 200.66 153.67 0)
 			(hide yes)
 			(show_name no)
@@
 		)
 		(property "Description" "Power symbol creates a global label with name \"GNDA\" , analog ground"
-			(at 200.66 157.48 0)
+			(at 200.66 153.67 0)
 			(hide yes)
 			(show_name no)
@@
 	(symbol
 		(lib_id "Device:C")
-		(at 190.5 157.48 90)
+		(at 190.5 153.67 90)
 		(unit 1)
 		(body_style 1)
@@
 		(fields_autoplaced yes)
 		(property "Reference" "C25"
-			(at 190.5 149.86 90)
+			(at 190.5 146.05 90)
 			(show_name no)
 			(do_not_autoplace no)
@@
 		)
 		(property "Value" "C"
-			(at 190.5 152.4 90)
+			(at 190.5 148.59 90)
 			(show_name no)
 			(do_not_autoplace no)
@@
 		)
 		(property "Footprint" ""
-			(at 194.31 156.5148 0)
+			(at 194.31 152.7048 0)
 			(hide yes)
 			(show_name no)
@@
 		)
 		(property "Datasheet" ""
-			(at 190.5 157.48 0)
+			(at 190.5 153.67 0)
 			(hide yes)
 			(show_name no)
@@
 		)
 		(property "Description" "Unpolarized capacitor"
-			(at 190.5 157.48 0)
+			(at 190.5 153.67 0)
 			(hide yes)
 			(show_name no)
@@
 		)
 	)
+	(embedded_fonts no)
 )
