File: OPA828_OUT.kicad_sch (KiCad schematic)
At the start: 4 parts, among them U1 OPA828ID

Commit message: main
Parts:
- renumbered C35 to C1, C37 to C2, C36 to C3, U1 to U7
Changed lines of the file:
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@@
-		)
-	)
-	(label "V_DAC_OUT"
-		(at 54.61 88.9 0)
-		(effects
-			(font
-				(size 1.27 1.27)
-			)
-			(justify left bottom)
 		)
 	)
@@
 			)
 			(justify left bottom)
+		)
+	)
+	(hierarchical_label "V_DAC_OUT"
+		(shape input)
+		(at 54.61 88.9 0)
+		(effects
+			(font
+				(size 1.27 1.27)
+			)
+			(justify left)
 		)
 	)
@@
 		(instances
 			(project "DAC11001"
-				(path "/d47dddaa-1169-4924-a666-b75ea4bc2aeb/97ba46ee-9723-4f8c-811a-5f0a70e859ab/66c60e08-9e27-4204-ab8d-ff51346a6bc8"
+				(path "/d47dddaa-1169-4924-a666-b75ea4bc2aeb/7933b1d9-37b7-42e4-861c-0c3dd9e959de"
 					(reference "#PWR035")
 					(unit 1)
@@
 		(dnp no)
 		(fields_autoplaced yes)
-		(property "Reference" "C36"
+		(property "Reference" "C3"
 			(at 152.4 76.2 90)
 			(show_name no)
@@
 		(instances
 			(project "DAC11001"
-				(path "/d47dddaa-1169-4924-a666-b75ea4bc2aeb/97ba46ee-9723-4f8c-811a-5f0a70e859ab/66c60e08-9e27-4204-ab8d-ff51346a6bc8"
-					(reference "C36")
+				(path "/d47dddaa-1169-4924-a666-b75ea4bc2aeb/7933b1d9-37b7-42e4-861c-0c3dd9e959de"
+					(reference "C3")
 					(unit 1)
 				)
@@
 		(instances
 			(project "DAC11001"
-				(path "/d47dddaa-1169-4924-a666-b75ea4bc2aeb/97ba46ee-9723-4f8c-811a-5f0a70e859ab/66c60e08-9e27-4204-ab8d-ff51346a6bc8"
+				(path "/d47dddaa-1169-4924-a666-b75ea4bc2aeb/7933b1d9-37b7-42e4-861c-0c3dd9e959de"
 					(reference "#PWR034")
 					(unit 1)
@@
 		(dnp no)
 		(fields_autoplaced yes)
-		(property "Reference" "U1"
+		(property "Reference" "U7"
 			(at 114.3 80.01 0)
 			(show_name no)
@@
 		(instances
 			(project "DAC11001"
-				(path "/d47dddaa-1169-4924-a666-b75ea4bc2aeb/97ba46ee-9723-4f8c-811a-5f0a70e859ab/66c60e08-9e27-4204-ab8d-ff51346a6bc8"
-					(reference "U1")
+				(path "/d47dddaa-1169-4924-a666-b75ea4bc2aeb/7933b1d9-37b7-42e4-861c-0c3dd9e959de"
+					(reference "U7")
 					(unit 1)
 				)
@@
 		(dnp no)
 		(fields_autoplaced yes)
-		(property "Reference" "C37"
+		(property "Reference" "C2"
 			(at 146.05 55.88 90)
 			(show_name no)
@@
 		(instances
 			(project "DAC11001"
-				(path "/d47dddaa-1169-4924-a666-b75ea4bc2aeb/97ba46ee-9723-4f8c-811a-5f0a70e859ab/66c60e08-9e27-4204-ab8d-ff51346a6bc8"
-					(reference "C37")
+				(path "/d47dddaa-1169-4924-a666-b75ea4bc2aeb/7933b1d9-37b7-42e4-861c-0c3dd9e959de"
+					(reference "C2")
 					(unit 1)
 				)
@@
 		(dnp no)
 		(fields_autoplaced yes)
-		(property "Reference" "C35"
+		(property "Reference" "C1"
 			(at 101.6 107.95 90)
 			(show_name no)
@@
 		(instances
 			(project "DAC11001"
-				(path "/d47dddaa-1169-4924-a666-b75ea4bc2aeb/97ba46ee-9723-4f8c-811a-5f0a70e859ab/66c60e08-9e27-4204-ab8d-ff51346a6bc8"
-					(reference "C35")
+				(path "/d47dddaa-1169-4924-a666-b75ea4bc2aeb/7933b1d9-37b7-42e4-861c-0c3dd9e959de"
+					(reference "C1")
 					(unit 1)
 				)

Commit message: modular
Connections:
- net V_C_+15V: no longer names the net of C3.1, U7.7 (V+)
- net V_FINAL_OUT renamed V_ROFS
Changed lines of the file:
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@@
+	(wire
+		(pts
+			(xy 81.28 62.23) (xy 81.28 67.31)
+		)
+		(stroke
+			(width 0)
+			(type default)
+		)
+	)
 	(wire
 		(pts
@@
 	(wire
 		(pts
+			(xy 83.82 49.53) (xy 83.82 54.61)
+		)
+		(stroke
+			(width 0)
+			(type default)
+		)
+	)
+	(wire
+		(pts
 			(xy 142.24 67.31) (xy 142.24 63.5)
 		)
@@
 	(wire
 		(pts
+			(xy 85.09 62.23) (xy 81.28 62.23)
+		)
+		(stroke
+			(width 0)
+			(type default)
+		)
+	)
+	(wire
+		(pts
 			(xy 54.61 88.9) (xy 54.61 95.25)
 		)
@@
 			(width 0)
 			(type default)
-		)
-	)
-	(label "V_ROFS"
-		(at 83.82 54.61 0)
-		(effects
-			(font
-				(size 1.27 1.27)
-			)
-			(justify left bottom)
-		)
-	)
-	(label "V_C_+15V"
-		(at 144.78 73.66 0)
-		(effects
-			(font
-				(size 1.27 1.27)
-			)
-			(justify left bottom)
 		)
 	)
@@
 		)
 	)
-	(label "V_RCM"
-		(at 81.28 67.31 0)
-		(effects
-			(font
-				(size 1.27 1.27)
-			)
-			(justify left bottom)
-		)
-	)
 	(label "V_C_-15"
 		(at 95.25 124.46 0)
@@
 			)
 			(justify left bottom)
+		)
+	)
+	(hierarchical_label "V_RCM"
+		(shape input)
+		(at 85.09 62.23 0)
+		(effects
+			(font
+				(size 1.27 1.27)
+			)
+			(justify left)
 		)
 	)
@@
 		(effects
 			(font
+				(size 1.27 1.27)
+			)
+			(justify left)
+		)
+	)
+	(hierarchical_label "V_ROFS"
+		(shape input)
+		(at 83.82 49.53 0)
+		(effects
+			(font

Commit message: main
Connections:
- net V_P_C_+15V: now reaches C3.1, U7.7 (V+)
- net V_C_-15 renamed V_P_C_-15V
Changed lines of the file:
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@@
 		)
 	)
-	(label "V_FINAL_OUT"
-		(at 207.01 95.25 0)
+	(label "V_P_C_+15V"
+		(at 144.78 73.66 0)
 		(effects
 			(font
@@
 		)
 	)
-	(label "V_C_-15"
+	(label "V_P_C_-15V"
 		(at 95.25 124.46 0)
 		(effects
 			(font
+				(size 1.27 1.27)
+			)
+			(justify left bottom)
+		)
+	)
+	(label "V_FINAL_OUT"
+		(at 207.01 95.25 0)
+		(effects
+			(font

Commit message: globaled
Connections:
- net V_ROFS renamed V_FINAL_OUT
Changed lines of the file:
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@@
 		)
 	)
-	(label "V_P_C_+15V"
-		(at 144.78 73.66 0)
+	(global_label "V_P_C_-15V"
+		(shape input)
+		(at 95.25 124.46 180)
+		(fields_autoplaced yes)
 		(effects
 			(font
 				(size 1.27 1.27)
 			)
-			(justify left bottom)
+			(justify right)
+		)
+		(property "Intersheetrefs" "${INTERSHEET_REFS}"
+			(at 80.6534 124.46 0)
+			(hide yes)
+			(show_name no)
+			(do_not_autoplace no)
+			(effects
+				(font
+					(size 1.27 1.27)
+				)
+				(justify right)
+			)
 		)
 	)
-	(label "V_P_C_-15V"
-		(at 95.25 124.46 0)
+	(global_label "V_P_C_+15V"
+		(shape input)
+		(at 144.78 73.66 180)
+		(fields_autoplaced yes)
 		(effects
 			(font
 				(size 1.27 1.27)
 			)
-			(justify left bottom)
+			(justify right)
+		)
+		(property "Intersheetrefs" "${INTERSHEET_REFS}"
+			(at 130.1834 73.66 0)
+			(hide yes)
+			(show_name no)
+			(do_not_autoplace no)
+			(effects
+				(font
+					(size 1.27 1.27)
+				)
+				(justify right)
+			)
 		)
 	)
-	(label "V_FINAL_OUT"
+	(global_label "V_FINAL_OUT"
+		(shape input)
 		(at 207.01 95.25 0)
+		(fields_autoplaced yes)
 		(effects
 			(font
 				(size 1.27 1.27)
 			)
-			(justify left bottom)
+			(justify left)
+		)
+		(property "Intersheetrefs" "${INTERSHEET_REFS}"
+			(at 221.7882 95.25 0)
+			(hide yes)
+			(show_name no)
+			(do_not_autoplace no)
+			(effects
+				(font
+					(size 1.27 1.27)
+				)
+				(justify left)
+			)
 		)
 	)
