File: DAC11001.kicad_sch (KiCad schematic)
At the start: 5 parts

Commit message: main
Connections:
- net V_C_+15V is gone; now on net V_P_REF_SENSE: DAC11001. (NC)
- net V_C_-15 is gone; now on net V_P_REF_SENSE: DAC11001. (NC)
- net V_DAC_OUT is gone; now on net V_P_REF_SENSE: DAC11001. (NC)
- new net LT3042/V_C_+15V: DAC11001. (NC)
- new net LT3094/V_C_-15V: DAC11001. (NC)
- new net OPA828 OUT/V_DAC_OUT: DAC11001. (NC)
Other:
- removed sheet +-15V Supply
- removed sheet Output Stage
- removed sheet Reference Voltages
- removed sheet SPI
- added sheet LT3042 (lt3042.kicad_sch)
- added sheet LT3094 (lt3094.kicad_sch)
- added sheet LTC3042v2 (LTC3042v2.kicad_sch)
- added sheet OPA828 OUT (OPA828_OUT.kicad_sch)
- moved on the sheet: DAC11001, R1, R18, R2, R3

Commit message: modular
Connections:
- net LT3042/V_C_+15V is gone; now on net V_P_C_-15V: DAC11001. (NC)
- net LT3094/V_C_-15V is gone; now on net V_P_C_-15V: DAC11001. (NC)
- net V_N_REF_FORCE is gone; now on net V_P_C_-15V: DAC11001. (NC)
- net V_N_REF_SENSE is gone; now on net V_P_C_-15V: DAC11001. (NC)
- net V_P_REF_FORCE is gone; now on net V_P_C_-15V: DAC11001. (NC)
- net V_P_REF_SENSE is gone; now on net V_P_C_-15V: DAC11001. (NC)
- net V_P_C_-15V: now reaches DAC11001. (NC)
- net V_RCM renamed OPA828 OUT/V_RCM
- net V_ROFS renamed OPA828 OUT/V_ROFS
- new net OPA828 4x/V_REF+_FORCE: DAC11001. (NC)
- new net OPA828 4x/V_REF+_SENSE: DAC11001. (NC)
- new net OPA828 4x/V_REF-_FORCE: DAC11001. (NC)
- new net OPA828 4x/V_REF-_SENSE: DAC11001. (NC)
- new net V_P_C_+15V: DAC11001. (NC)
Other:
- removed sheet LT3042
- removed sheet LT3094
- removed sheet LTC3042v2
- added sheet OPA828 4x (opa828_4x.kicad_sch)
- sheet OPA828 OUT ports: added V_RCM, V_ROFS; removed none
- moved on the sheet: R1

Commit message: done
Connections:
- net CLR is gone; now on net V_P_C_-15V: DAC11001. (NC)
- net LDAC is gone; now on net V_P_C_-15V: DAC11001. (NC)
- net SCLK is gone; now on net V_P_C_-15V: DAC11001. (NC)
- net SDIN is gone; now on net V_P_C_-15V: DAC11001. (NC)
- net SDO is gone; now on net V_P_C_-15V: DAC11001. (NC)
- net SYNC is gone; now on net V_P_C_-15V: DAC11001. (NC)
- new net ISO7761/CLR: DAC11001. (NC)
- new net ISO7761/LDAC: DAC11001. (NC)
- new net ISO7761/SCLK: DAC11001. (NC)
- new net ISO7761/SDIN: DAC11001. (NC)
- new net ISO7761/SDO: DAC11001. (NC)
- new net ISO7761/SYNC: DAC11001. (NC)
Other:
- added sheet ISO7761 (iso.kicad_sch)
- moved on the sheet: DAC11001, R1, R18, R2, R3

Commit message: main
Connections:
- net 5V is gone; now on net V_P_C_-15V: DAC11001. (NC)
- new net V_P_5+: DAC11001. (NC)
Other:
- added sheet LT3042 (lt3042.kicad_sch)
- added sheet LT3042v2 (lt3042v2.kicad_sch)
- added sheet LT3042v3 (lt3042v3.kicad_sch)
- added sheet LT3094 (lt3094.kicad_sch)
- added sheet LT3999 (lt3999.kicad_sch)
Changed lines of the file:
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@@
-		)
-	)
-	(label "5V"
-		(at 196.85 26.67 0)
-		(effects
-			(font
-				(size 1.27 1.27)
-			)
-			(justify left bottom)
 		)
 	)
@@
 		)
 	)
+	(label "V_P_5+"
+		(at 196.85 26.67 0)
+		(effects
+			(font
+				(size 1.27 1.27)
+			)
+			(justify left bottom)
+		)
+	)
 	(label "V_P_C_-15V"
 		(at 93.98 22.86 0)
@@
 	)
 	(sheet
-		(at 71.12 60.96)
-		(size 27.94 29.21)
+		(at 22.86 157.48)
+		(size 12.7 3.81)
 		(exclude_from_sim no)
 		(in_bom yes)
@@
 			(color 0 0 0 0)
 		)
+		(property "Sheetname" "LT3094"
+			(at 22.86 156.7684 0)
+			(show_name no)
+			(do_not_autoplace no)
+			(effects
+				(font
+					(size 1.27 1.27)
+				)
+				(justify left bottom)
+			)
+		)
+		(property "Sheetfile" "lt3094.kicad_sch"
+			(at 22.86 161.8746 0)
+			(show_name no)
+			(do_not_autoplace no)
+			(effects
+				(font
+					(size 1.27 1.27)
+				)
+				(justify left top)
+			)
+		)
+		(instances
+			(project "DAC11001"
+				(path "/d47dddaa-1169-4924-a666-b75ea4bc2aeb"
+					(page "11")
+				)
+			)
+		)
+	)
+	(sheet
+		(at 22.86 167.64)
+		(size 12.7 3.81)
+		(exclude_from_sim no)
+		(in_bom yes)
+		(on_board yes)
+		(dnp no)
+		(fields_autoplaced yes)
+		(stroke
+			(width 0.1524)
+			(type solid)
+		)
+		(fill
+			(color 0 0 0 0)
+		)
+		(property "Sheetname" "LT3042"
+			(at 22.86 166.9284 0)
+			(show_name no)
+			(do_not_autoplace no)
+			(effects
+				(font
+					(size 1.27 1.27)
+				)
+				(justify left bottom)
+			)
+		)
+		(property "Sheetfile" "lt3042.kicad_sch"
+			(at 22.86 172.0346 0)
+			(show_name no)
+			(do_not_autoplace no)
+			(effects
+				(font
+					(size 1.27 1.27)
+				)
+				(justify left top)
+			)
+		)
+		(instances
+			(project "DAC11001"
+				(path "/d47dddaa-1169-4924-a666-b75ea4bc2aeb"
+					(page "10")
+				)
+			)
+		)
+	)
+	(sheet
+		(at 71.12 60.96)
+		(size 27.94 29.21)
+		(exclude_from_sim no)
+		(in_bom yes)
+		(on_board yes)
+		(dnp no)
+		(fields_autoplaced yes)
+		(stroke
+			(width 0.1524)
+			(type solid)
+		)
+		(fill
+			(color 0 0 0 0)
+		)
 		(property "Sheetname" "OPA828 4x"
 			(at 71.12 60.2484 0)
@@
 				)
 			)
+		)
+	)
+	(sheet
+		(at 53.34 157.48)
+		(size 12.7 3.81)
+		(exclude_from_sim no)
+		(in_bom yes)
+		(on_board yes)
+		(dnp no)
+		(fields_autoplaced yes)
+		(stroke
+			(width 0.1524)
+			(type solid)
+		)
+		(fill
+			(color 0 0 0 0)
+		)
+		(property "Sheetname" "LT3042v2"
+			(at 53.34 156.7684 0)
+			(show_name no)
+			(do_not_autoplace no)
+			(effects
+				(font
+					(size 1.27 1.27)
+				)
+				(justify left bottom)
+			)
+		)
+		(property "Sheetfile" "lt3042v2.kicad_sch"
+			(at 53.34 161.8746 0)
+			(show_name no)
+			(do_not_autoplace no)
+			(effects
+				(font
+					(size 1.27 1.27)
+				)
+				(justify left top)
+			)
+		)
+		(instances
+			(project "DAC11001"
+				(path "/d47dddaa-1169-4924-a666-b75ea4bc2aeb"
+					(page "13")
+				)
+			)
+		)
+	)
+	(sheet
+		(at 55.88 171.45)
+		(size 12.7 3.81)
+		(exclude_from_sim no)
+		(in_bom yes)
+		(on_board yes)
+		(dnp no)
+		(fields_autoplaced yes)
+		(stroke
+			(width 0.1524)
+			(type solid)
+		)
+		(fill
+			(color 0 0 0 0)
+		)
+		(property "Sheetname" "LT3042v3"
+			(at 55.88 170.7384 0)
+			(show_name no)
+			(do_not_autoplace no)
+			(effects
+				(font
+					(size 1.27 1.27)
+				)
+				(justify left bottom)
+			)
+		)
+		(property "Sheetfile" "lt3042v3.kicad_sch"
+			(at 55.88 175.8446 0)
+			(show_name no)
+			(do_not_autoplace no)
+			(effects
+				(font
+					(size 1.27 1.27)
+				)
+				(justify left top)
+			)
+		)
+		(instances
+			(project "DAC11001"
+				(path "/d47dddaa-1169-4924-a666-b75ea4bc2aeb"
+					(page "14")
+				)
+			)
+		)
+	)
+	(sheet
+		(at 22.86 177.8)
+		(size 12.7 3.81)
+		(exclude_from_sim no)
+		(in_bom yes)
+		(on_board yes)
+		(dnp no)
+		(fields_autoplaced yes)
+		(stroke
+			(width 0.1524)
+			(type solid)
+		)
+		(fill
+			(color 0 0 0 0)
+		)
+		(property "Sheetname" "LT3999"
+			(at 22.86 177.0884 0)
+			(show_name no)
+			(do_not_autoplace no)
+			(effects
+				(font
+					(size 1.27 1.27)
+				)
+				(justify left bottom)
+			)
+		)
+		(property "Sheetfile" "lt3999.kicad_sch"
+			(at 22.86 182.1946 0)
+			(show_name no)
+			(do_not_autoplace no)
+			(effects
+				(font
+					(size 1.27 1.27)
+				)
+				(justify left top)
+			)
+		)
+		(instances
+			(project "DAC11001"
+				(path "/d47dddaa-1169-4924-a666-b75ea4bc2aeb"
+					(page "7")
+				)
+			)

Commit message: globaled
Other:
- removed sheet LT3042
- removed sheet LT3042v2
- removed sheet LT3042v3
- removed sheet LT3094
- removed sheet LT3999
Changed lines of the file:
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@@
 	(paper "A4")
+	(junction
+		(at 190.5 26.67)
+		(diameter 0)
+		(color 0 0 0 0)
+	)
 	(junction
 		(at 163.83 40.64)
@@
 	)
 	(junction
-		(at 190.5 26.67)
-		(diameter 0)
-		(color 0 0 0 0)
-	)
-	(junction
 		(at 186.69 143.51)
 		(diameter 0)
@@
 	(wire
 		(pts
-			(xy 196.85 26.67) (xy 190.5 26.67)
+			(xy 201.93 26.67) (xy 190.5 26.67)
 		)
 		(stroke
@@
 		)
 	)
-	(label "V_P_C_+15V"
-		(at 93.98 27.94 0)
+	(global_label "V_P_C_-15V"
+		(shape input)
+		(at 93.98 22.86 180)
+		(fields_autoplaced yes)
 		(effects
 			(font
 				(size 1.27 1.27)
 			)
-			(justify left bottom)
-		)
-	)
-	(label "V_P_5+"
-		(at 196.85 26.67 0)
+			(justify right)
+		)
+		(property "Intersheetrefs" "${INTERSHEET_REFS}"
+			(at 79.3834 22.86 0)
+			(hide yes)
+			(show_name no)
+			(do_not_autoplace no)
+			(effects
+				(font
+					(size 1.27 1.27)
+				)
+				(justify right)
+			)
+		)
+	)
+	(global_label "V_P_C_+15V"
+		(shape input)
+		(at 93.98 27.94 180)
+		(fields_autoplaced yes)
 		(effects
 			(font
 				(size 1.27 1.27)
 			)
-			(justify left bottom)
-		)
-	)
-	(label "V_P_C_-15V"
-		(at 93.98 22.86 0)
+			(justify right)
+		)
+		(property "Intersheetrefs" "${INTERSHEET_REFS}"
+			(at 79.3834 27.94 0)
+			(hide yes)
+			(show_name no)
+			(do_not_autoplace no)
+			(effects
+				(font
+					(size 1.27 1.27)
+				)
+				(justify right)
+			)
+		)
+	)
+	(global_label "V_P_5+"
+		(shape input)
+		(at 201.93 26.67 0)
+		(fields_autoplaced yes)
 		(effects
 			(font
 				(size 1.27 1.27)
 			)
-			(justify left bottom)
+			(justify left)
+		)
+		(property "Intersheetrefs" "${INTERSHEET_REFS}"
+			(at 211.9909 26.67 0)
+			(hide yes)
+			(show_name no)
+			(do_not_autoplace no)
+			(effects
+				(font
+					(size 1.27 1.27)
+				)
+				(justify left)
+			)
 		)
 	)
@@
 	)
 	(sheet
-		(at 22.86 157.48)
-		(size 12.7 3.81)
-		(exclude_from_sim no)
-		(in_bom yes)
-		(on_board yes)
-		(dnp no)
-		(fields_autoplaced yes)
-		(stroke
-			(width 0.1524)
-			(type solid)
-		)
-		(fill
-			(color 0 0 0 0)
-		)
-		(property "Sheetname" "LT3094"
-			(at 22.86 156.7684 0)
-			(show_name no)
-			(do_not_autoplace no)
-			(effects
-				(font
-					(size 1.27 1.27)
-				)
-				(justify left bottom)
-			)
-		)
-		(property "Sheetfile" "lt3094.kicad_sch"
-			(at 22.86 161.8746 0)
-			(show_name no)
-			(do_not_autoplace no)
-			(effects
-				(font
-					(size 1.27 1.27)
-				)
-				(justify left top)
-			)
-		)
-		(instances
-			(project "DAC11001"
-				(path "/d47dddaa-1169-4924-a666-b75ea4bc2aeb"
-					(page "11")
-				)
-			)
-		)
-	)
-	(sheet
-		(at 22.86 167.64)
-		(size 12.7 3.81)
-		(exclude_from_sim no)
-		(in_bom yes)
-		(on_board yes)
-		(dnp no)
-		(fields_autoplaced yes)
-		(stroke
-			(width 0.1524)
-			(type solid)
-		)
-		(fill
-			(color 0 0 0 0)
-		)
-		(property "Sheetname" "LT3042"
-			(at 22.86 166.9284 0)
-			(show_name no)
-			(do_not_autoplace no)
-			(effects
-				(font
-					(size 1.27 1.27)
-				)
-				(justify left bottom)
-			)
-		)
-		(property "Sheetfile" "lt3042.kicad_sch"
-			(at 22.86 172.0346 0)
-			(show_name no)
-			(do_not_autoplace no)
-			(effects
-				(font
-					(size 1.27 1.27)
-				)
-				(justify left top)
-			)
-		)
-		(instances
-			(project "DAC11001"
-				(path "/d47dddaa-1169-4924-a666-b75ea4bc2aeb"
-					(page "10")
-				)
-			)
-		)
-	)
-	(sheet
 		(at 71.12 60.96)
 		(size 27.94 29.21)
@@
 				)
 			)
-		)
-	)
-	(sheet
-		(at 53.34 157.48)
-		(size 12.7 3.81)
-		(exclude_from_sim no)
-		(in_bom yes)
-		(on_board yes)
-		(dnp no)
-		(fields_autoplaced yes)
-		(stroke
-			(width 0.1524)
-			(type solid)
-		)
-		(fill
-			(color 0 0 0 0)
-		)
-		(property "Sheetname" "LT3042v2"
-			(at 53.34 156.7684 0)
-			(show_name no)
-			(do_not_autoplace no)
-			(effects
-				(font
-					(size 1.27 1.27)
-				)
-				(justify left bottom)
-			)
-		)
-		(property "Sheetfile" "lt3042v2.kicad_sch"
-			(at 53.34 161.8746 0)
-			(show_name no)
-			(do_not_autoplace no)
-			(effects
-				(font
-					(size 1.27 1.27)
-				)
-				(justify left top)
-			)
-		)
-		(instances
-			(project "DAC11001"
-				(path "/d47dddaa-1169-4924-a666-b75ea4bc2aeb"
-					(page "13")
-				)
-			)
-		)
-	)
-	(sheet
-		(at 55.88 171.45)
-		(size 12.7 3.81)
-		(exclude_from_sim no)
-		(in_bom yes)
-		(on_board yes)
-		(dnp no)
-		(fields_autoplaced yes)
-		(stroke
-			(width 0.1524)
-			(type solid)
-		)
-		(fill
-			(color 0 0 0 0)
-		)
-		(property "Sheetname" "LT3042v3"
-			(at 55.88 170.7384 0)
-			(show_name no)
-			(do_not_autoplace no)
-			(effects
-				(font
-					(size 1.27 1.27)
-				)
-				(justify left bottom)
-			)
-		)
-		(property "Sheetfile" "lt3042v3.kicad_sch"
-			(at 55.88 175.8446 0)
-			(show_name no)
-			(do_not_autoplace no)
-			(effects
-				(font
-					(size 1.27 1.27)
-				)
-				(justify left top)
-			)
-		)
-		(instances
-			(project "DAC11001"
-				(path "/d47dddaa-1169-4924-a666-b75ea4bc2aeb"
-					(page "14")
-				)
-			)
-		)
-	)
-	(sheet
-		(at 22.86 177.8)
-		(size 12.7 3.81)
-		(exclude_from_sim no)
-		(in_bom yes)
-		(on_board yes)
-		(dnp no)
-		(fields_autoplaced yes)
-		(stroke
-			(width 0.1524)
-			(type solid)
-		)
-		(fill
-			(color 0 0 0 0)
-		)
-		(property "Sheetname" "LT3999"
-			(at 22.86 177.0884 0)
-			(show_name no)
-			(do_not_autoplace no)
-			(effects
-				(font
-					(size 1.27 1.27)
-				)
-				(justify left bottom)
-			)
-		)
-		(property "Sheetfile" "lt3999.kicad_sch"
-			(at 22.86 182.1946 0)
-			(show_name no)
-			(do_not_autoplace no)
-			(effects
-				(font
-					(size 1.27 1.27)
-				)
-				(justify left top)
-			)
-		)
-		(instances
-			(project "DAC11001"
-				(path "/d47dddaa-1169-4924-a666-b75ea4bc2aeb"
-					(page "7")
-				)
-			)

Commit message: done
Other:
- added sheet LT3999 (lt3999.kicad_sch)
Changed lines of the file:
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@@
+		)
+	)
+	(sheet
+		(at 35.56 148.59)
+		(size 43.18 16.51)
+		(exclude_from_sim no)
+		(in_bom yes)
+		(on_board yes)
+		(dnp no)
+		(fields_autoplaced yes)
+		(stroke
+			(width 0.1524)
+			(type solid)
+		)
+		(fill
+			(color 0 0 0 0)
+		)
+		(property "Sheetname" "LT3999"
+			(at 35.56 147.8784 0)
+			(show_name no)
+			(do_not_autoplace no)
+			(effects
+				(font
+					(size 1.27 1.27)
+				)
+				(justify left bottom)
+			)
+		)
+		(property "Sheetfile" "lt3999.kicad_sch"
+			(at 35.56 165.6846 0)
+			(show_name no)
+			(do_not_autoplace no)
+			(effects
+				(font
+					(size 1.27 1.27)
+				)
+				(justify left top)
+			)
+		)
+		(instances
+			(project "DAC11001"
+				(path "/d47dddaa-1169-4924-a666-b75ea4bc2aeb"
+					(page "6")
+				)
+			)
 		)
 	)
