File: lt3042v3.kicad_sch (KiCad schematic)
At the start: 8 parts, among them U4 LT3094MPDD-PBF

Commit message: main
Parts:
- removed C7, C8, C9: C, symbol Device:C
- removed R10, R11, R8, R9: R, symbol Device:R
- removed U4: LT3094MPDD-PBF, DD_05-08-1725_ADI, symbol 2026-06-29_19-42-13:LT3094MPDD-PBF
- added C35, C36, C39: C, symbol Device:C
- added R35, R36, R37, R38: R, symbol Device:R
- added U9: LT3042EDD-PBF, DFN-10_DD_LIT, symbol 2026-06-29_19-42-44:LT3042EDD-PBF
Connections:
- net GND: now also C35.2, C36.2, C39.2, R35.2, R36.2, R38.2, U9.11 (GND), U9.8 (GND)
- new net: R35.1, U9.5 (ILIM)
- new net: R37.2, R38.1, U9.6 (PGFB)
- new net: C36.1, R36.1, U9.7 (SET)
- new net V_P_+12V: C35.1, U9.1 (IN), U9.2 (IN), U9.3 (EN/UV)
- new net V_P_5+: C39.1, R37.1, U9.10 (OUT), U9.9 (OUTS)

Commit message: globaled
Changed lines of the file:
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@@
 		)
 	)
-	(label "V_P_5+"
-		(at 243.84 78.74 0)
+	(global_label "V_P_+12V"
+		(shape input)
+		(at 52.07 76.2 180)
+		(fields_autoplaced yes)
 		(effects
 			(font
 				(size 1.27 1.27)
 			)
-			(justify left bottom)
-		)
-	)
-	(label "V_P_+12V"
-		(at 52.07 76.2 0)
+			(justify right)
+		)
+		(property "Intersheetrefs" "${INTERSHEET_REFS}"
+			(at 39.711 76.2 0)
+			(hide yes)
+			(show_name no)
+			(do_not_autoplace no)
+			(effects
+				(font
+					(size 1.27 1.27)
+				)
+				(justify right)
+			)
+		)
+	)
+	(global_label "V_P_5+"
+		(shape input)
+		(at 243.84 78.74 0)
+		(fields_autoplaced yes)
 		(effects
 			(font
 				(size 1.27 1.27)
 			)
-			(justify left bottom)
+			(justify left)
+		)
+		(property "Intersheetrefs" "${INTERSHEET_REFS}"
+			(at 253.9009 78.74 0)
+			(hide yes)
+			(show_name no)
+			(do_not_autoplace no)
+			(effects
+				(font
+					(size 1.27 1.27)
+				)
+				(justify left)
+			)
 		)
 	)
@@
 				)
 			)
-			(project "DAC11001"
-				(path "/d47dddaa-1169-4924-a666-b75ea4bc2aeb/b4e2e048-73d5-47b9-a078-31dc77393363"
-					(reference "U17")
-					(unit 1)
-				)
-			)
 		)
 	)
@@
 				)
 			)
-			(project "DAC11001"
-				(path "/d47dddaa-1169-4924-a666-b75ea4bc2aeb/b4e2e048-73d5-47b9-a078-31dc77393363"
-					(reference "C49")
-					(unit 1)
-				)
-			)
 		)
 	)
@@
 				)
 			)
-			(project "DAC11001"
-				(path "/d47dddaa-1169-4924-a666-b75ea4bc2aeb/b4e2e048-73d5-47b9-a078-31dc77393363"
-					(reference "#PWR039")
-					(unit 1)
-				)
-			)
 		)
 	)
@@
 				)
 			)
-			(project "DAC11001"
-				(path "/d47dddaa-1169-4924-a666-b75ea4bc2aeb/b4e2e048-73d5-47b9-a078-31dc77393363"
-					(reference "C51")
-					(unit 1)
-				)
-			)
 		)
 	)
@@
 				)
 			)
-			(project "DAC11001"
-				(path "/d47dddaa-1169-4924-a666-b75ea4bc2aeb/b4e2e048-73d5-47b9-a078-31dc77393363"
-					(reference "R56")
-					(unit 1)
-				)
-			)
 		)
 	)
@@
 				)
 			)
-			(project "DAC11001"
-				(path "/d47dddaa-1169-4924-a666-b75ea4bc2aeb/b4e2e048-73d5-47b9-a078-31dc77393363"
-					(reference "R57")
-					(unit 1)
-				)
-			)
 		)
 	)
@@
 				)
 			)
-			(project "DAC11001"
-				(path "/d47dddaa-1169-4924-a666-b75ea4bc2aeb/b4e2e048-73d5-47b9-a078-31dc77393363"
-					(reference "C50")
-					(unit 1)
-				)
-			)
 		)
 	)
@@
 				)
 			)
-			(project "DAC11001"
-				(path "/d47dddaa-1169-4924-a666-b75ea4bc2aeb/b4e2e048-73d5-47b9-a078-31dc77393363"
-					(reference "R58")
-					(unit 1)
-				)
-			)
 		)
 	)
@@
 					(unit 1)
 				)
-			)
-			(project "DAC11001"
-				(path "/d47dddaa-1169-4924-a666-b75ea4bc2aeb/b4e2e048-73d5-47b9-a078-31dc77393363"
-					(reference "R55")
-					(unit 1)
-				)

Commit message: done
Parts:
- renumbered C35 to C51, C36 to C54, C39 to C55, R35 to R59, R36 to R63, R37 to R64, R38 to R65, U9 to U19
Changed lines of the file:
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@@
 		(dnp no)
 		(fields_autoplaced yes)
-		(property "Reference" "U9"
+		(property "Reference" "U19"
 			(at 135.89 66.04 0)
 			(show_name no)
@@
 		(instances
 			(project "DAC11001"
+				(path "/688e2b68-3871-489b-b27a-c18d3c11fcf6/9763c458-ad2a-49f6-b267-7cfd74c6fed3/b2d57cbb-ac61-46e7-a525-a854f0e63ea1"
+					(reference "U10")
+					(unit 1)
+				)
+			)
+			(project "DAC11001"
 				(path "/7fba4707-d072-468a-a501-14a80bae184d"
 					(reference "U9")
+					(unit 1)
+				)
+			)
+			(project ""
+				(path "/abdba638-bc95-4869-83fe-bbcdf8030f26/b2d57cbb-ac61-46e7-a525-a854f0e63ea1"
+					(reference "U9")
+					(unit 1)
+				)
+			)
+			(project "DAC11001"
+				(path "/d47dddaa-1169-4924-a666-b75ea4bc2aeb/a8da5177-43c4-4665-b682-d49b9fc3d5b2/9763c458-ad2a-49f6-b267-7cfd74c6fed3/b2d57cbb-ac61-46e7-a525-a854f0e63ea1"
+					(reference "U19")
 					(unit 1)
 				)
@@
 		(dnp no)
 		(fields_autoplaced yes)
-		(property "Reference" "C35"
+		(property "Reference" "C51"
 			(at 82.55 78.7399 0)
 			(show_name no)
@@
 		(instances
 			(project "DAC11001"
+				(path "/688e2b68-3871-489b-b27a-c18d3c11fcf6/9763c458-ad2a-49f6-b267-7cfd74c6fed3/b2d57cbb-ac61-46e7-a525-a854f0e63ea1"
+					(reference "C42")
+					(unit 1)
+				)
+			)
+			(project "DAC11001"
 				(path "/7fba4707-d072-468a-a501-14a80bae184d"
 					(reference "C35")
+					(unit 1)
+				)
+			)
+			(project ""
+				(path "/abdba638-bc95-4869-83fe-bbcdf8030f26/b2d57cbb-ac61-46e7-a525-a854f0e63ea1"
+					(reference "C35")
+					(unit 1)
+				)
+			)
+			(project "DAC11001"
+				(path "/d47dddaa-1169-4924-a666-b75ea4bc2aeb/a8da5177-43c4-4665-b682-d49b9fc3d5b2/9763c458-ad2a-49f6-b267-7cfd74c6fed3/b2d57cbb-ac61-46e7-a525-a854f0e63ea1"
+					(reference "C51")
 					(unit 1)
 				)
@@
 		(instances
 			(project "DAC11001"
+				(path "/688e2b68-3871-489b-b27a-c18d3c11fcf6/9763c458-ad2a-49f6-b267-7cfd74c6fed3/b2d57cbb-ac61-46e7-a525-a854f0e63ea1"
+					(reference "#PWR039")
+					(unit 1)
+				)
+			)
+			(project "DAC11001"
 				(path "/7fba4707-d072-468a-a501-14a80bae184d"
+					(reference "#PWR039")
+					(unit 1)
+				)
+			)
+			(project ""
+				(path "/abdba638-bc95-4869-83fe-bbcdf8030f26/b2d57cbb-ac61-46e7-a525-a854f0e63ea1"
+					(reference "#PWR039")
+					(unit 1)
+				)
+			)
+			(project "DAC11001"
+				(path "/d47dddaa-1169-4924-a666-b75ea4bc2aeb/a8da5177-43c4-4665-b682-d49b9fc3d5b2/9763c458-ad2a-49f6-b267-7cfd74c6fed3/b2d57cbb-ac61-46e7-a525-a854f0e63ea1"
 					(reference "#PWR039")
 					(unit 1)
@@
 		(dnp no)
 		(fields_autoplaced yes)
-		(property "Reference" "C39"
+		(property "Reference" "C55"
 			(at 219.71 91.4399 0)
 			(show_name no)
@@
 		(instances
 			(project "DAC11001"
+				(path "/688e2b68-3871-489b-b27a-c18d3c11fcf6/9763c458-ad2a-49f6-b267-7cfd74c6fed3/b2d57cbb-ac61-46e7-a525-a854f0e63ea1"
+					(reference "C44")
+					(unit 1)
+				)
+			)
+			(project "DAC11001"
 				(path "/7fba4707-d072-468a-a501-14a80bae184d"
 					(reference "C39")
+					(unit 1)
+				)
+			)
+			(project ""
+				(path "/abdba638-bc95-4869-83fe-bbcdf8030f26/b2d57cbb-ac61-46e7-a525-a854f0e63ea1"
+					(reference "C39")
+					(unit 1)
+				)
+			)
+			(project "DAC11001"
+				(path "/d47dddaa-1169-4924-a666-b75ea4bc2aeb/a8da5177-43c4-4665-b682-d49b9fc3d5b2/9763c458-ad2a-49f6-b267-7cfd74c6fed3/b2d57cbb-ac61-46e7-a525-a854f0e63ea1"
+					(reference "C55")
 					(unit 1)
 				)
@@
 		(dnp no)
 		(fields_autoplaced yes)
-		(property "Reference" "R36"
+		(property "Reference" "R63"
 			(at 179.07 99.0599 0)
 			(show_name no)
@@
 		(instances
 			(project "DAC11001"
+				(path "/688e2b68-3871-489b-b27a-c18d3c11fcf6/9763c458-ad2a-49f6-b267-7cfd74c6fed3/b2d57cbb-ac61-46e7-a525-a854f0e63ea1"
+					(reference "R44")
+					(unit 1)
+				)
+			)
+			(project "DAC11001"
 				(path "/7fba4707-d072-468a-a501-14a80bae184d"
 					(reference "R36")
+					(unit 1)
+				)
+			)
+			(project ""
+				(path "/abdba638-bc95-4869-83fe-bbcdf8030f26/b2d57cbb-ac61-46e7-a525-a854f0e63ea1"
+					(reference "R36")
+					(unit 1)
+				)
+			)
+			(project "DAC11001"
+				(path "/d47dddaa-1169-4924-a666-b75ea4bc2aeb/a8da5177-43c4-4665-b682-d49b9fc3d5b2/9763c458-ad2a-49f6-b267-7cfd74c6fed3/b2d57cbb-ac61-46e7-a525-a854f0e63ea1"
+					(reference "R63")
 					(unit 1)
 				)
@@
 		(dnp no)
 		(fields_autoplaced yes)
-		(property "Reference" "R37"
+		(property "Reference" "R64"
 			(at 203.2 83.8199 0)
 			(show_name no)
@@
 		(instances
 			(project "DAC11001"
+				(path "/688e2b68-3871-489b-b27a-c18d3c11fcf6/9763c458-ad2a-49f6-b267-7cfd74c6fed3/b2d57cbb-ac61-46e7-a525-a854f0e63ea1"
+					(reference "R45")
+					(unit 1)
+				)
+			)
+			(project "DAC11001"
 				(path "/7fba4707-d072-468a-a501-14a80bae184d"
 					(reference "R37")
+					(unit 1)
+				)
+			)
+			(project ""
+				(path "/abdba638-bc95-4869-83fe-bbcdf8030f26/b2d57cbb-ac61-46e7-a525-a854f0e63ea1"
+					(reference "R37")
+					(unit 1)
+				)
+			)
+			(project "DAC11001"
+				(path "/d47dddaa-1169-4924-a666-b75ea4bc2aeb/a8da5177-43c4-4665-b682-d49b9fc3d5b2/9763c458-ad2a-49f6-b267-7cfd74c6fed3/b2d57cbb-ac61-46e7-a525-a854f0e63ea1"
+					(reference "R64")
 					(unit 1)
 				)
@@
 		(dnp no)
 		(fields_autoplaced yes)
-		(property "Reference" "C36"
+		(property "Reference" "C54"
 			(at 171.45 99.0599 0)
 			(show_name no)
@@
 		(instances
 			(project "DAC11001"
+				(path "/688e2b68-3871-489b-b27a-c18d3c11fcf6/9763c458-ad2a-49f6-b267-7cfd74c6fed3/b2d57cbb-ac61-46e7-a525-a854f0e63ea1"
+					(reference "C43")
+					(unit 1)
+				)
+			)
+			(project "DAC11001"
 				(path "/7fba4707-d072-468a-a501-14a80bae184d"
 					(reference "C36")
+					(unit 1)
+				)
+			)
+			(project ""
+				(path "/abdba638-bc95-4869-83fe-bbcdf8030f26/b2d57cbb-ac61-46e7-a525-a854f0e63ea1"
+					(reference "C36")
+					(unit 1)
+				)
+			)
+			(project "DAC11001"
+				(path "/d47dddaa-1169-4924-a666-b75ea4bc2aeb/a8da5177-43c4-4665-b682-d49b9fc3d5b2/9763c458-ad2a-49f6-b267-7cfd74c6fed3/b2d57cbb-ac61-46e7-a525-a854f0e63ea1"
+					(reference "C54")
 					(unit 1)
 				)
@@
 		(dnp no)
 		(fields_autoplaced yes)
-		(property "Reference" "R38"
+		(property "Reference" "R65"
 			(at 203.2 93.9799 0)
 			(show_name no)
@@
 		(instances
 			(project "DAC11001"
+				(path "/688e2b68-3871-489b-b27a-c18d3c11fcf6/9763c458-ad2a-49f6-b267-7cfd74c6fed3/b2d57cbb-ac61-46e7-a525-a854f0e63ea1"
+					(reference "R46")
+					(unit 1)
+				)
+			)
+			(project "DAC11001"
 				(path "/7fba4707-d072-468a-a501-14a80bae184d"
 					(reference "R38")
+					(unit 1)
+				)
+			)
+			(project ""
+				(path "/abdba638-bc95-4869-83fe-bbcdf8030f26/b2d57cbb-ac61-46e7-a525-a854f0e63ea1"
+					(reference "R38")
+					(unit 1)
+				)
+			)
+			(project "DAC11001"
+				(path "/d47dddaa-1169-4924-a666-b75ea4bc2aeb/a8da5177-43c4-4665-b682-d49b9fc3d5b2/9763c458-ad2a-49f6-b267-7cfd74c6fed3/b2d57cbb-ac61-46e7-a525-a854f0e63ea1"
+					(reference "R65")
 					(unit 1)
 				)
@@
 		(dnp no)
 		(fields_autoplaced yes)
-		(property "Reference" "R35"
+		(property "Reference" "R59"
 			(at 107.95 100.3299 0)
 			(show_name no)
@@
 		(instances
 			(project "DAC11001"
+				(path "/688e2b68-3871-489b-b27a-c18d3c11fcf6/9763c458-ad2a-49f6-b267-7cfd74c6fed3/b2d57cbb-ac61-46e7-a525-a854f0e63ea1"
+					(reference "R43")
+					(unit 1)
+				)
+			)
+			(project "DAC11001"
 				(path "/7fba4707-d072-468a-a501-14a80bae184d"
 					(reference "R35")
 					(unit 1)
 				)
+			)
+			(project ""
+				(path "/abdba638-bc95-4869-83fe-bbcdf8030f26/b2d57cbb-ac61-46e7-a525-a854f0e63ea1"
+					(reference "R35")
+					(unit 1)
+				)
+			)
+			(project "DAC11001"
+				(path "/d47dddaa-1169-4924-a666-b75ea4bc2aeb/a8da5177-43c4-4665-b682-d49b9fc3d5b2/9763c458-ad2a-49f6-b267-7cfd74c6fed3/b2d57cbb-ac61-46e7-a525-a854f0e63ea1"
+					(reference "R59")
+					(unit 1)
+				)
